File: emg_dsp/stage4/dual_amp.sch (KiCad schematic (older format))
At the start: 4 parts, among them U47 LMV1032, U48 LMV1032, U49 LMV1032

Commit message: oops, forgot to add in the new amp sub-schematic.
Parts:
- removed C87: 0.047uf, 0402, symbol C
- added U? (x4): C2, 0405, symbol C2
- added U? (x2): LMV1032-25, microSMD-4, symbol LMV1032
- added U?: LMV1032-15, microSMD-4, symbol LMV1032
- U47, U48: value LMV1032 -> LMV1032-25
- U49: value LMV1032 -> LMV1032-15
Connections:
- net labels added: in0, in1, out0, out1
- net labels removed: in, out
- wire segments 13 -> 32
Other:
- note added: "capacitor to ground on the output"
- note added: "causes instability. bad idea!"
- note removed: "15db"
- note removed: "25db"
- moved on the sheet: U48, U49
Changed lines of the file:
@@
-EESchema Schematic File Version 2  date Thu 28 Jan 2010 05:31:53 PM EST
+EESchema Schematic File Version 2  date Sun 31 Jan 2010 07:35:14 PM EST
 LIBS:power,device,emg_sym,./stage4.cache
 EELAYER 24  0
 EELAYER END
 $Descr A4 11700 8267
-Sheet 5 39
+Sheet 39 39
 Title ""
 Date "9 jan 2009"
@@
 Comment4 ""
 $EndDescr
-Text HLabel 5750 4050 2    60   Input ~ 0
+Connection ~ 4300 3800
+Wire Wire Line
+	4300 3800 4300 4500
+Wire Wire Line
+	4300 4500 4200 4500
+Connection ~ 7100 3800
+Wire Wire Line
+	7100 3800 7100 4500
+Wire Wire Line
+	7100 4500 7000 4500
+Connection ~ 6250 4050
+Wire Wire Line
+	6250 4050 6250 4500
+Wire Wire Line
+	6250 4500 6350 4500
+Connection ~ 3550 4050
+Wire Wire Line
+	7500 4050 3450 4050
+Wire Wire Line
+	3450 4050 3450 4500
+Wire Wire Line
+	3450 4500 3550 4500
+Connection ~ 7000 3800
+Wire Wire Line
+	7000 3350 7000 3800
+Connection ~ 4950 4050
+Wire Wire Line
+	4950 3350 4950 4050
+Wire Wire Line
+	5600 3200 5650 3200
+Wire Wire Line
+	4200 3200 4250 3200
+Wire Wire Line
+	3550 4050 3550 3350
+Wire Wire Line
+	4200 3350 4200 3800
+Wire Wire Line
+	3550 3200 3400 3200
+Wire Wire Line
+	4900 3200 4950 3200
+Wire Wire Line
+	6300 3200 6350 3200
+Wire Wire Line
+	4200 3800 7500 3800
+Wire Wire Line
+	6350 3350 6350 4050
+Connection ~ 6350 4050
+Wire Wire Line
+	5600 3350 5600 3800
+Connection ~ 5600 3800
+Wire Wire Line
+	7000 3200 7500 3200
+Wire Wire Line
+	5600 4350 5650 4350
+Wire Wire Line
+	4200 4350 4250 4350
+Wire Wire Line
+	3550 4350 3400 4350
+Wire Wire Line
+	4900 4350 4950 4350
+Wire Wire Line
+	6300 4350 6350 4350
+Wire Wire Line
+	7000 4350 7500 4350
+Wire Wire Line
+	4950 4500 4850 4500
+Wire Wire Line
+	4850 4500 4850 4050
+Connection ~ 4850 4050
+Wire Wire Line
+	5600 4500 5700 4500
+Wire Wire Line
+	5700 4500 5700 3800
+Connection ~ 5700 3800
+$Comp
+L C2 U?
+U 2 1 4B662126
+P 5950 4350
+F 0 "U?" H 6000 4200 60  0000 C CNN
+F 1 "C2" H 6000 4500 60  0000 C CNN
+F 2 "0405" H 6000 4050 60  0000 C CNN
+	2    5950 4350
+	1    0    0    -1
+$EndComp
+$Comp
+L C2 U?
+U 2 1 4B662125
+P 4550 4350
+F 0 "U?" H 4600 4200 60  0000 C CNN
+F 1 "C2" H 4600 4500 60  0000 C CNN
+F 2 "0405" H 4600 4050 60  0000 C CNN
+	2    4550 4350
+	1    0    0    -1
+$EndComp
+Text HLabel 3400 4350 0    60   Input ~ 0
+in1
+Text HLabel 7500 4350 2    60   Input ~ 0
+out1
+$Comp
+L LMV1032 U?
+U 1 1 4B662124
+P 6700 4400
+F 0 "U?" H 6700 4100 60  0000 C CNN
+F 1 "LMV1032-15" H 6700 4200 60  0000 C CNN
+F 2 "microSMD-4" H 6640 4040 60  0000 C CNN
+	1    6700 4400
+	-1   0    0    -1
+$EndComp
+$Comp
+L LMV1032 U?
+U 1 1 4B662123
+P 5300 4400
+F 0 "U?" H 5300 4100 60  0000 C CNN
+F 1 "LMV1032-25" H 5300 4200 60  0000 C CNN
+F 2 "microSMD-4" H 5240 4040 60  0000 C CNN
+	1    5300 4400
+	-1   0    0    -1
+$EndComp
+$Comp
+L LMV1032 U?
+U 1 1 4B662122
+P 3900 4400
+F 0 "U?" H 3900 4100 60  0000 C CNN
+F 1 "LMV1032-25" H 3900 4200 60  0000 C CNN
+F 2 "microSMD-4" H 3840 4040 60  0000 C CNN
+	1    3900 4400
+	-1   0    0    -1
+$EndComp
+$Comp
+L C2 U?
+U 1 1 4B6620F6
+P 5950 3200
+F 0 "U?" H 6000 3050 60  0000 C CNN
+F 1 "C2" H 6000 3350 60  0000 C CNN
+F 2 "0405" H 6000 2900 60  0000 C CNN
+	1    5950 3200
+	1    0    0    -1
+$EndComp
+$Comp
+L C2 U?
+U 1 1 4B6620D9
+P 4550 3200
+F 0 "U?" H 4600 3050 60  0000 C CNN
+F 1 "C2" H 4600 3350 60  0000 C CNN
+F 2 "0405" H 4600 2900 60  0000 C CNN
+	1    4550 3200
+	1    0    0    -1
+$EndComp
+Text Notes 7150 3500 0    60   ~ 0
+causes instability.  bad idea!
+Text Notes 7150 3400 0    60   ~ 0
+capacitor to ground on the output
+Text HLabel 7500 4050 2    60   Input ~ 0
 Vdd
-Text HLabel 6750 3800 2    60   Input ~ 0
+Text HLabel 7500 3800 2    60   Input ~ 0
 GND
-Text Notes 5950 3100 0    60   ~ 0
-25db
-Text Notes 4900 3100 0    60   ~ 0
-25db
-Text Notes 3700 3100 0    60   ~ 0
-15db
-Wire Wire Line
-	3550 3200 3400 3200
-Wire Wire Line
-	6750 3600 6750 3800
-Wire Wire Line
-	6750 3800 4200 3800
-Connection ~ 4700 4050
-Wire Wire Line
-	5750 3350 5750 4050
-Wire Wire Line
-	5750 4050 3550 4050
-Connection ~ 5350 3800
-Wire Wire Line
-	6400 3800 6400 3350
-Wire Wire Line
-	5350 3200 5750 3200
-Wire Wire Line
-	4200 3200 4700 3200
-Wire Wire Line
-	4200 3800 4200 3350
-Wire Wire Line
-	5350 3800 5350 3350
-Wire Wire Line
-	3550 4050 3550 3350
-Wire Wire Line
-	4700 4050 4700 3350
-Connection ~ 6750 3200
-Connection ~ 6400 3800
-Wire Wire Line
-	7200 3200 6400 3200
 Text HLabel 3400 3200 0    60   Input ~ 0
-in
-Text HLabel 7200 3200 2    60   Input ~ 0
-out
-$Comp
-L C C87
-U 1 1 48C9FE70
-P 6750 3400
-AR Path="/48C9FDD8/48C9FE11/48C9FE70" Ref="C87"  Part="1"
-AR Path="/48C9FDD8/48CA00FF/48C9FE70" Ref="C118"  Part="1"
-AR Path="/48C9FDD8/48CA00FE/48C9FE70" Ref="C117"  Part="1"
-AR Path="/48C9FDD8/48CA00FD/48C9FE70" Ref="C116"  Part="1"
-AR Path="/48C9FDD8/48CA00FC/48C9FE70" Ref="C115"  Part="1"
-AR Path="/48C9FDD8/48CA00FB/48C9FE70" Ref="C114"  Part="1"
-AR Path="/48C9FDD8/48CA00FA/48C9FE70" Ref="C113"  Part="1"
-AR Path="/48C9FDD8/48CA00F9/48C9FE70" Ref="C112"  Part="1"
-AR Path="/48C9FDD8/48CA00F8/48C9FE70" Ref="C111"  Part="1"
-AR Path="/48C9FDD8/48CA00F7/48C9FE70" Ref="C110"  Part="1"
-AR Path="/48C9FDD8/48CA00F6/48C9FE70" Ref="C109"  Part="1"
-AR Path="/48C9FDD8/48CA00F5/48C9FE70" Ref="C108"  Part="1"
-AR Path="/48C9FDD8/48CA00F4/48C9FE70" Ref="C107"  Part="1"
-AR Path="/48C9FDD8/48CA00F3/48C9FE70" Ref="C106"  Part="1"
-AR Path="/48C9FDD8/48CA00F2/48C9FE70" Ref="C105"  Part="1"
-AR Path="/48C9FDD8/48CA00F1/48C9FE70" Ref="C104"  Part="1"
-AR Path="/48C9FDD8/48CA00F0/48C9FE70" Ref="C103"  Part="1"
-AR Path="/48C9FDD8/48CA00CF/48C9FE70" Ref="C102"  Part="1"
-AR Path="/48C9FDD8/48CA00CE/48C9FE70" Ref="C101"  Part="1"
-AR Path="/48C9FDD8/48CA00CD/48C9FE70" Ref="C100"  Part="1"
-AR Path="/48C9FDD8/48CA00CC/48C9FE70" Ref="C99"  Part="1"
-AR Path="/48C9FDD8/48CA00CB/48C9FE70" Ref="C98"  Part="1"
-AR Path="/48C9FDD8/48CA00CA/48C9FE70" Ref="C97"  Part="1"
-AR Path="/48C9FDD8/48CA00C9/48C9FE70" Ref="C96"  Part="1"
-AR Path="/48C9FDD8/48CA00C8/48C9FE70" Ref="C95"  Part="1"
-AR Path="/48C9FDD8/48CA00A7/48C9FE70" Ref="C94"  Part="1"
-AR Path="/48C9FDD8/48CA00A6/48C9FE70" Ref="C93"  Part="1"
-AR Path="/48C9FDD8/48CA00A5/48C9FE70" Ref="C92"  Part="1"
-AR Path="/48C9FDD8/48CA00A4/48C9FE70" Ref="C91"  Part="1"
-AR Path="/48C9FDD8/48CA008E/48C9FE70" Ref="C90"  Part="1"
-AR Path="/48C9FDD8/48CA007D/48C9FE70" Ref="C89"  Part="1"
-AR Path="/48C9FDD8/48CA002F/48C9FE70" Ref="C88"  Part="1"
-F 0 "C88" H 6800 3500 50  0000 L CNN
-F 1 "0.047uf" H 6800 3300 50  0000 L CNN
-F 2 "0402" H 6950 3200 60  0000 C CNN
-	1    6750 3400
-	1    0    0    -1
-$EndComp
+in0
+Text HLabel 7500 3200 2    60   Input ~ 0
+out0
 $Comp
 L LMV1032 U49
 U 1 1 48C9FE5C
-P 6100 3250
+P 6700 3250
 AR Path="/48C9FDD8/48C9FE11/48C9FE5C" Ref="U49"  Part="1"
 AR Path="/48C9FDD8/48CA00FF/48C9FE5C" Ref="U142"  Part="1"
@@
 AR Path="/48C9FDD8/48CA007D/48C9FE5C" Ref="U55"  Part="1"
 AR Path="/48C9FDD8/48CA002F/48C9FE5C" Ref="U52"  Part="1"
-F 0 "U52" H 6100 2950 60  0000 C CNN
-F 1 "LMV1032" H 6100 3050 60  0000 C CNN
-F 2 "microSMD-4" H 6040 2890 60  0000 C CNN
-	1    6100 3250
+F 0 "U49" H 6700 2950 60  0000 C CNN
+F 1 "LMV1032-15" H 6700 3050 60  0000 C CNN
+F 2 "microSMD-4" H 6640 2890 60  0000 C CNN
+	1    6700 3250
 	-1   0    0    -1
 $EndComp
@@
 L LMV1032 U48
 U 1 1 48C9FE4D
-P 5050 3250
+P 5300 3250
 AR Path="/48C9FDD8/48C9FE11/48C9FE4D" Ref="U48"  Part="1"
 AR Path="/48C9FDD8/48CA00FF/48C9FE4D" Ref="U141"  Part="1"
@@
 AR Path="/48C9FDD8/48CA007D/48C9FE4D" Ref="U54"  Part="1"
 AR Path="/48C9FDD8/48CA002F/48C9FE4D" Ref="U51"  Part="1"
-F 0 "U51" H 5050 2950 60  0000 C CNN
-F 1 "LMV1032" H 5050 3050 60  0000 C CNN
-F 2 "microSMD-4" H 4990 2890 60  0000 C CNN
-	1    5050 3250
+F 0 "U48" H 5300 2950 60  0000 C CNN
+F 1 "LMV1032-25" H 5300 3050 60  0000 C CNN
+F 2 "microSMD-4" H 5240 2890 60  0000 C CNN
+	1    5300 3250
 	-1   0    0    -1
 $EndComp
@@
 AR Path="/48C9FDD8/48CA007D/48C9FE38" Ref="U53"  Part="1"
 AR Path="/48C9FDD8/48CA002F/48C9FE38" Ref="U50"  Part="1"
-F 0 "U50" H 3900 2950 60  0000 C CNN
-F 1 "LMV1032" H 3900 3050 60  0000 C CNN
+F 0 "U47" H 3900 2950 60  0000 C CNN
+F 1 "LMV1032-25" H 3900 3050 60  0000 C CNN
 F 2 "microSMD-4" H 3840 2890 60  0000 C CNN
 	1    3900 3250
