File: emg_dsp/stage4/stage2_analog.sch (KiCad schematic (older format))
At the start: 30 parts, among them U145 OMNETICS_36, U24 ADG726, U25 JUMP, U26 TPS71727, U27 TPS71727, U28 THS4281, U29 THS4281, U30 ADCS7476, U31 ADCS7476

Commit message: added the active electrode - just an INA, opamp, highpass and two lowpasses.
Parts:
- removed TP?: TP, TP, symbol TP
- added R? (x2): 3.3k, 0402, symbol R
- added R? (x2): 1.5k, 0402, symbol R
- added R?: 100k, 0402, symbol R
- added TP?: TP, TP, symbol TP
Connections:
- wire segments 230 -> 227
Other:
- note added: "dnp if not using AFE"
- moved on the sheet: TP?

Commit message: revamping the neural AFE
Connections:
- net labels added: A16, A17, A18, A19, A20, A21, A22, A23, A24, A25, A26, A27, A28, A29, A30, A31, mux0, mux1, mux2, mux3
- net labels removed: B0, B1, B10, B11, B12, B13, B14, B15, B2, B3, B4, B5, B6, B7, B8, B9
- wire segments 227 -> 280
Other:
- note added: "not sure if this will"
- note added: "work ok at 2.7V.."

Commit message: nearing completion for stage4!
Parts:
- removed C55: 2.2uf, 0402, symbol C
- added C? (x2): 0.1uf, 0402, symbol C
- added C?: 2.2uf, 0402, symbol C
- added R?: 20, 0402, symbol R
- added R?: 40k, 0402, symbol R
- added TP? (x3): TP, TP, symbol TP
- added U?: 74HC4067BQ, VQFN-24, symbol 74HC4067
- added U? (x3): LMV1032-25, microSMD-4, symbol LMV1032
- added U?: JUMP, 2x100mil, symbol JUMP
- C56, C57, C58: value 0.012uf -> 0.1uf
Connections:
- wire segments 280 -> 305
Other:
- note added: "for measuring the noise charateristics of the amps."

Commit message: getting closer to finalizing the schematic ... added another voltage, beh.
Parts:
- removed C56, C58: 0.1uf, 0402, symbol C
- removed C62: 2.2uf, 0402, symbol C
- removed C66: 0.012uf, 0402, symbol C
- removed L7: INDUCTOR, 0603, symbol INDUCTOR
- removed R?: 100k, 0402, symbol R
- removed U25: JUMP, 2x100mil, symbol JUMP
- removed U27: TPS71727, SC-70-5, symbol TPS717
- added C? (x2): 0.1uf, 0402, symbol C
- added C? (x2): 1uf, 0402, symbol C
- added C? (x2): 2.2uf, 0402, symbol C
- added C?: 0.012uf, 0402, symbol C
- added L? (x2): ferrite, 0402, symbol INDUCTOR
- added U? (x3): JUMP, 2x100mil, symbol JUMP
- added U?: TPS71718, SC-70-5, symbol TPS717
Connections:
- net labels added: V18, V27, VAA, VDD
- net labels removed: AFEEN, V27A, V27B, VIN
- wire segments 305 -> 307
Other:
- note added: "supply your own voltage!"
- moved on the sheet: C53, C57, C61, C65, TP?, U26

Commit message: fixing the schematic with the help of the BOM.. trying to make the BOM simpler (and also making sure that U can actually buy all the parts on the board!)
Parts:
- removed C57, C?: 0.1uf, 0402, symbol C
- added C66: 2.2uf, 0402, symbol C
- added U35: MUX_VDD, 2x100mil, symbol JUMP
- C70: renamed from C53; value 2.2uf -> 1uf
- C71: renamed from C?; value 2.2uf -> 1uf
- C78: renamed from C65; value 0.012uf -> 0.01uf
- C79: renamed from C?; value 0.012uf -> 0.01uf
- R46: renamed from R?; value 40k -> 50k
- R47: renamed from R?; value 20 -> 25
- TP26: renamed from TP?; value TP -> MUX_A
- TP27: renamed from TP?; value TP -> MUX_B
- TP28: renamed from TP?; value TP -> T1
- TP29: renamed from TP?; value TP -> T2
- TP30: renamed from TP?; value TP -> T3
- U33: renamed from U?; value JUMP -> EN_V27
- U34: renamed from U?; value JUMP -> EN_V18
- U44: renamed from U?; value JUMP -> TEST_SIG
- U47: renamed from U?; value JUMP -> TEST_SPLY
- U48: renamed from U?; value LMV1032-25 -> LMV1032-15
- gave numbers to parts that had none: 17
- renumbered C49 to C62, C50 to C63, C51 to C64, C52 to C65, C54 to C67, C59 to C72, C60 to C73, C63 to C74, C64 to C75, C61 to C76, U24 to U36, U28 to U37, U29 to U38, U26 to U39, U30 to U41, U31 to U42, U145 to U43
Connections:
- wire segments 307 -> 312
Other:
- note added: "3.3V?"
- note added: "on resistance may be too high"
- moved on the sheet: C76, C77, C78, C79, U32, U39, U40
