File: emg_dsp/stage4/microstim4.sch (KiCad schematic (older format))
At the start: 34 parts, among them U64 10X100, U65 6533-CONN, U66 SW_DPDT, U67 5.5MMJACK, U68 DCV01, U69 GND, U70 EN_BF, U71 74HC245, U72 MAX3004, U73 EN_DAQ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

Commit message: cleaned up the power supplies.  not sure what i was thinking before - 2.85V should be fine for Vdd.
Other:
- note added: "2.85V"
- note removed: "2.85/3.3V"

Commit message: layout 95% done ...
Parts:
- removed C115: 0.1uf, 0603, symbol C
Other:
- moved on the sheet: C118
Changed lines of the file:
@@
-EESchema Schematic File Version 2  date Fri 19 Feb 2010 01:29:26 AM EST
+EESchema Schematic File Version 2  date Mon 22 Feb 2010 06:59:14 PM EST
 LIBS:power,device,emg_sym,/home/tlh24/svn/myopen/emg_dsp/lib/linear,./stage4.cache
 EELAYER 24  0
@@
 L VEE #PWR237
 U 1 1 4B68CC05
-P 8100 6600
-F 0 "#PWR237" H 8100 6800 40  0001 C CNN
-F 1 "VEE" H 8100 6750 40  0000 C CNN
-	1    8100 6600
-	1    0    0    -1
-$EndComp
-$Comp
-L VEE #PWR223
-U 1 1 4B68CC02
 P 6150 6550
-F 0 "#PWR223" H 6150 6750 40  0001 C CNN
+F 0 "#PWR237" H 6150 6750 40  0001 C CNN
 F 1 "VEE" H 6150 6700 40  0000 C CNN
 	1    6150 6550
@@
 $Comp
 L GND #PWR0146
-U 1 1 47F01B3F
-P 6150 6950
-F 0 "#PWR0146" H 6150 6950 30  0001 C CNN
-F 1 "GND" H 6150 6880 30  0001 C CNN
-	1    6150 6950
-	1    0    0    -1
-$EndComp
-$Comp
-L C C115
-U 1 1 47F01B3D
-P 6150 6750
-F 0 "C115" H 6200 6850 50  0000 L CNN
-F 1 "0.1uf" H 6200 6650 50  0000 L CNN
-F 2 "0603" H 6000 6850 60  0000 C CNN
-	1    6150 6750
-	1    0    0    -1
-$EndComp
-$Comp
-L GND #PWR0147
 U 1 1 47F01B2A
 P 5650 6400
-F 0 "#PWR0147" H 5650 6400 30  0001 C CNN
+F 0 "#PWR0146" H 5650 6400 30  0001 C CNN
 F 1 "GND" H 5650 6330 30  0001 C CNN
 	1    5650 6400
@@
 $EndComp
 $Comp
-L GND #PWR0148
+L GND #PWR0147
 U 1 1 47F002CE
-P 8100 7000
-F 0 "#PWR0148" H 8100 7000 30  0001 C CNN
-F 1 "GND" H 8100 6930 30  0001 C CNN
-	1    8100 7000
+P 6150 6950
+F 0 "#PWR0147" H 6150 6950 30  0001 C CNN
+F 1 "GND" H 6150 6880 30  0001 C CNN
+	1    6150 6950
 	1    0    0    -1
 $EndComp
@@
 L C C118
 U 1 1 47F002B2
-P 8100 6800
-F 0 "C118" H 8150 6900 50  0000 L CNN
-F 1 "0.1uf" H 8150 6700 50  0000 L CNN
-F 2 "0603" H 7950 6900 60  0000 C CNN
-	1    8100 6800
-	1    0    0    -1
-$EndComp
+P 6150 6750
+F 0 "C118" H 6200 6850 50  0000 L CNN
+F 1 "0.1uf" H 6200 6650 50  0000 L CNN
+F 2 "0603" H 6000 6850 60  0000 C CNN
+	1    6150 6750
+	1    0    0    -1
+$EndComp

Commit message: it's zone time~!
Connections:
- wire segments 210 -> 214
Changed lines of the file:
@@
-EESchema Schematic File Version 2  date Mon 22 Feb 2010 06:59:14 PM EST
+EESchema Schematic File Version 2  date Tue 23 Feb 2010 01:51:22 PM EST
 LIBS:power,device,emg_sym,/home/tlh24/svn/myopen/emg_dsp/lib/linear,./stage4.cache
 EELAYER 24  0
@@
 Comment4 ""
 $EndDescr
-Text Notes 5700 750  0    60   ~ 0
-cannels arrayed at 1.1"
+$Comp
+L GND #PWR?
+U 1 1 4B84239B
+P 1950 4600
+F 0 "#PWR?" H 1950 4600 30  0001 C CNN
+F 1 "GND" H 1950 4530 30  0001 C CNN
+	1    1950 4600
+	1    0    0    -1
+$EndComp
+Connection ~ 1950 4550
+Wire Wire Line
+	1950 4550 1950 4600
 Wire Wire Line
 	9150 3000 8550 3000
@@
 Wire Wire Line
 	9150 2900 8550 2900
+Wire Wire Line
+	1850 4450 1850 4550
+Wire Wire Line
+	1850 4550 2050 4550
+Wire Wire Line
+	2050 4550 2050 4450
+Text Notes 5700 750  0    60   ~ 0
+cannels arrayed at 1.1"
 $Comp
 L TP TP49
@@
 _cs1-4
 $Comp
-L GND #PWR0118
+L GND #PWR0120
 U 1 1 4B68C1BF
 P 7600 3650
-F 0 "#PWR0118" H 7600 3650 30  0001 C CNN
+F 0 "#PWR0120" H 7600 3650 30  0001 C CNN
 F 1 "GND" H 7600 3580 30  0001 C CNN
 	1    7600 3650
@@
 PPI8
 $Comp
-L GND #PWR0119
+L GND #PWR0121
 U 1 1 4B68C137
 P 8700 4400
-F 0 "#PWR0119" H 8700 4400 30  0001 C CNN
+F 0 "#PWR0121" H 8700 4400 30  0001 C CNN
 F 1 "GND" H 8700 4330 30  0001 C CNN
 	1    8700 4400
@@
 $EndComp
 $Comp
-L GND #PWR0120
+L GND #PWR0122
 U 1 1 4B68C134
 P 7700 4450
-F 0 "#PWR0120" H 7700 4450 30  0001 C CNN
+F 0 "#PWR0122" H 7700 4450 30  0001 C CNN
 F 1 "GND" H 7700 4380 30  0001 C CNN
 	1    7700 4450
@@
 $EndComp
 $Comp
-L VDD #PWR0121
+L VDD #PWR0123
 U 1 1 4B68C133
 P 7700 4050
-F 0 "#PWR0121" H 7700 4150 30  0001 C CNN
+F 0 "#PWR0123" H 7700 4150 30  0001 C CNN
 F 1 "VDD" H 7700 4160 30  0000 C CNN
 	1    7700 4050
@@
 $EndComp
 $Comp
-L GND #PWR0122
+L GND #PWR0124
 U 1 1 4B68C131
 P 8550 3850
-F 0 "#PWR0122" H 8550 3850 30  0001 C CNN
+F 0 "#PWR0124" H 8550 3850 30  0001 C CNN
 F 1 "GND" H 8550 3780 30  0001 C CNN
 	1    8550 3850
@@
 $EndComp
 $Comp
-L VDD #PWR0123
+L VDD #PWR0125
 U 1 1 4B68C130
 P 7750 2700
-F 0 "#PWR0123" H 7750 2800 30  0001 C CNN
+F 0 "#PWR0125" H 7750 2800 30  0001 C CNN
 F 1 "VDD" H 7750 2810 30  0000 C CNN
 	1    7750 2700
@@
 a1
 $Comp
-L GND #PWR0124
+L GND #PWR0126
 U 1 1 4B68C0A1
 P 7150 4450
-F 0 "#PWR0124" H 7150 4450 30  0001 C CNN
+F 0 "#PWR0126" H 7150 4450 30  0001 C CNN
 F 1 "GND" H 7150 4380 30  0001 C CNN
 	1    7150 4450
@@
 $EndComp
 $Comp
-L GND #PWR0125
+L GND #PWR0127
 U 1 1 4B68C099
 P 5800 4550
-F 0 "#PWR0125" H 5800 4550 30  0001 C CNN
+F 0 "#PWR0127" H 5800 4550 30  0001 C CNN
 F 1 "GND" H 5800 4480 30  0001 C CNN
 	1    5800 4550
@@
 $EndComp
 $Comp
-L VDD #PWR0126
+L VDD #PWR0128
 U 1 1 4B68C098
 P 5800 4150
-F 0 "#PWR0126" H 5800 4250 30  0001 C CNN
+F 0 "#PWR0128" H 5800 4250 30  0001 C CNN
 F 1 "VDD" H 5800 4260 30  0000 C CNN
 	1    5800 4150
@@
 $EndComp
 $Comp
-L GND #PWR0127
+L GND #PWR0129
 U 1 1 4B68C07F
 P 6950 3850
-F 0 "#PWR0127" H 6950 3850 30  0001 C CNN
+F 0 "#PWR0129" H 6950 3850 30  0001 C CNN
 F 1 "GND" H 6950 3780 30  0001 C CNN
 	1    6950 3850
@@
 $EndComp
 $Comp
-L VDD #PWR0128
+L VDD #PWR0130
 U 1 1 4B68C05E
 P 6150 2700
-F 0 "#PWR0128" H 6150 2800 30  0001 C CNN
+F 0 "#PWR0130" H 6150 2800 30  0001 C CNN
 F 1 "VDD" H 6150 2810 30  0000 C CNN
 	1    6150 2700
@@
 PPI0
 $Comp
-L GND #PWR0129
+L GND #PWR0131
 U 1 1 4B68BF6C
 P 6150 4350
-F 0 "#PWR0129" H 6150 4350 30  0001 C CNN
+F 0 "#PWR0131" H 6150 4350 30  0001 C CNN
 F 1 "GND" H 6150 4280 30  0001 C CNN
 	1    6150 4350
@@
 NoConn ~ 1650 5650
 $Comp
-L GND #PWR0130
+L GND #PWR0132
 U 1 1 4A8AF09D
 P 3150 5650
-F 0 "#PWR0130" H 3150 5650 30  0001 C CNN
+F 0 "#PWR0132" H 3150 5650 30  0001 C CNN
 F 1 "GND" H 3150 5580 30  0001 C CNN
 	1    3150 5650
@@
 $EndComp
 $Comp
-L GND #PWR0131
+L GND #PWR0133
 U 1 1 4A8AF03C
 P 850 1900
-F 0 "#PWR0131" H 850 1900 30  0001 C CNN
+F 0 "#PWR0133" H 850 1900 30  0001 C CNN
 F 1 "GND" H 850 1830 30  0001 C CNN
 	1    850  1900
@@
 $EndComp
 $Comp
-L GND #PWR0132
+L GND #PWR0134
 U 1 1 4A8AF036
 P 850 900
-F 0 "#PWR0132" H 850 900 30  0001 C CNN
+F 0 "#PWR0134" H 850 900 30  0001 C CNN
 F 1 "GND" H 850 830 30  0001 C CNN
 	1    850  900
@@
 $EndComp
 $Comp
-L GND #PWR0133
+L GND #PWR0135
 U 1 1 49E368BC
 P 850 4400
-F 0 "#PWR0133" H 850 4400 30  0001 C CNN
+F 0 "#PWR0135" H 850 4400 30  0001 C CNN
 F 1 "GND" H 850 4330 30  0001 C CNN
 	1    850  4400
@@
 $EndComp
 $Comp
-L GND #PWR0134
+L GND #PWR0136
 U 1 1 49E368B8
 P 3050 4350
-F 0 "#PWR0134" H 3050 4350 30  0001 C CNN
+F 0 "#PWR0136" H 3050 4350 30  0001 C CNN
 F 1 "GND" H 3050 4280 30  0001 C CNN
 	1    3050 4350
@@
 $EndComp
 $Comp
-L GND #PWR0135
+L GND #PWR0137
 U 1 1 49D24134
 P 4500 5950
-F 0 "#PWR0135" H 4500 5950 30  0001 C CNN
+F 0 "#PWR0137" H 4500 5950 30  0001 C CNN
 F 1 "GND" H 4500 5880 30  0001 C CNN
 	1    4500 5950
@@
 NoConn ~ 2450 6700
 $Comp
-L GND #PWR0136
+L GND #PWR0138
 U 1 1 47F1AF0C
 P 2600 6650
-F 0 "#PWR0136" H 2600 6650 30  0001 C CNN
+F 0 "#PWR0138" H 2600 6650 30  0001 C CNN
 F 1 "GND" H 2600 6580 30  0001 C CNN
 	1    2600 6650
@@
 NoConn ~ 6550 5850
 $Comp
-L GND #PWR0137
+L GND #PWR0139
 U 1 1 47F1A8C3
 P 7050 5450
-F 0 "#PWR0137" H 7050 5450 30  0001 C CNN
+F 0 "#PWR0139" H 7050 5450 30  0001 C CNN
 F 1 "GND" H 7050 5380 30  0001 C CNN
 	1    7050 5450
@@
 NoConn ~ 2550 3100
 $Comp
-L GND #PWR0138
+L GND #PWR0140
 U 1 1 47F16634
 P 2900 6250
-F 0 "#PWR0138" H 2900 6250 30  0001 C CNN
+F 0 "#PWR0140" H 2900 6250 30  0001 C CNN
 F 1 "GND" H 2900 6180 30  0001 C CNN
 	1    2900 6250
@@
 $EndComp
 $Comp
-L GND #PWR0139
+L GND #PWR0141
 U 1 1 47F16605
 P 2600 7650
-F 0 "#PWR0139" H 2600 7650 30  0001 C CNN
+F 0 "#PWR0141" H 2600 7650 30  0001 C CNN
 F 1 "GND" H 2600 7580 30  0001 C CNN
 	1    2600 7650
@@
 _csin
 $Comp
-L GND #PWR0140
+L GND #PWR0142
 U 1 1 47F15728
 P 10500 6250
-F 0 "#PWR0140" H 10500 6250 30  0001 C CNN
+F 0 "#PWR0142" H 10500 6250 30  0001 C CNN
 F 1 "GND" H 10500 6180 30  0001 C CNN
 	1    10500 6250
@@
 $EndComp
 $Comp
-L GND #PWR0141
+L GND #PWR0143
 U 1 1 47F15727
 P 9300 5350
-F 0 "#PWR0141" H 9300 5350 30  0001 C CNN
+F 0 "#PWR0143" H 9300 5350 30  0001 C CNN
 F 1 "GND" H 9300 5280 30  0001 C CNN
 	1    9300 5350
@@
 c1
 $Comp
-L GND #PWR0142
+L GND #PWR0144
 U 1 1 47F15566
 P 1250 7000
-F 0 "#PWR0142" H 1250 7000 30  0001 C CNN
+F 0 "#PWR0144" H 1250 7000 30  0001 C CNN
 F 1 "GND" H 1250 6930 30  0001 C CNN
 	1    1250 7000
@@
 NoConn ~ 1650 5550
 $Comp
-L GND #PWR0143
+L GND #PWR0145
 U 1 1 47F068CF
 P 1400 5500
-F 0 "#PWR0143" H 1400 5500 30  0001 C CNN
+F 0 "#PWR0145" H 1400 5500 30  0001 C CNN
 F 1 "GND" H 1400 5430 30  0001 C CNN
 	1    1400 5500
@@
 _csin
 $Comp
-L GND #PWR0144
+L GND #PWR0146
 U 1 1 47F01EE5
 P 8700 6250
-F 0 "#PWR0144" H 8700 6250 30  0001 C CNN
+F 0 "#PWR0146" H 8700 6250 30  0001 C CNN
 F 1 "GND" H 8700 6180 30  0001 C CNN
 	1    8700 6250
@@
 $EndComp
 $Comp
-L GND #PWR0145
+L GND #PWR0147
 U 1 1 47F01EA9
 P 7500 5350
-F 0 "#PWR0145" H 7500 5350 30  0001 C CNN
+F 0 "#PWR0147" H 7500 5350 30  0001 C CNN
 F 1 "GND" H 7500 5280 30  0001 C CNN
 	1    7500 5350
@@
 _csin
 $Comp
-L GND #PWR0146
+L GND #PWR0148
 U 1 1 47F01B2A
 P 5650 6400
-F 0 "#PWR0146" H 5650 6400 30  0001 C CNN
+F 0 "#PWR0148" H 5650 6400 30  0001 C CNN
 F 1 "GND" H 5650 6330 30  0001 C CNN
 	1    5650 6400
@@
 $EndComp
 $Comp
-L GND #PWR0147
+L GND #PWR0149
 U 1 1 47F002CE
 P 6150 6950
-F 0 "#PWR0147" H 6150 6950 30  0001 C CNN
+F 0 "#PWR0149" H 6150 6950 30  0001 C CNN
 F 1 "GND" H 6150 6880 30  0001 C CNN
 	1    6150 6950
