File: emg_dsp/stage5/active_electrode2.sch (KiCad schematic (older format))
At the start: 27 parts, among them U1 MAX4208, U2 LMV321

Commit message: I think I'm going to need to array the active electrodes manually - then can put some other stuff on the board too.  woohoo.
Other:
- note added: "lp @ 3.2kHz"
- note removed: "hp @ 3.2kHz"
Changed lines of the file:
@@
-EESchema Schematic File Version 2  date Mon 19 Apr 2010 01:17:39 PM EDT
+EESchema Schematic File Version 2  date Mon 19 Apr 2010 02:46:26 PM EDT
 LIBS:power,device,emg_sym,/home/tlh24/svn/myopen/emg_dsp/lib/linear
 EELAYER 24  0
@@
 	6200 3550 6350 3550
 Text Notes 5250 2850 0    60   ~ 0
-hp @ 3.2kHz
+lp @ 3.2kHz
 $Comp
 L ZENER D2
