File: emg_dsp/stage5/stage5.sch (KiCad schematic (older format))
At the start: 162 parts, among them U1 TPS71733, U10 TPS62410, U11 FCI_USB_B, U13 VCC_1.2, U15 EN_VCC, U17 EN_VDD, U2 ADM3202, U21 ABM10XTAL, U22 BF532-160, U24 NRF24L01, U26 74LCX541, U27 MAX6711Z, U28 TESTCON, U29 ANTENNA, U3 MAX3421E, U30 74LCX541, U5 VEE, U6 ADSP_JTAG_CON, U7 NX3225SA, U9 RS232_CON

Commit message: working on stage5 already -- will it be tight?
Parts:
- added C32: 0.1uf, 0402, symbol C
- added U8: GT12MABE, GT12MABE, symbol GT12MABE
- gave numbers to parts that had none: 49
- renumbered C14 to C10, C17 to C11, C19 to C12, C8 to C13, C21 to C14, C11 to C15, C23 to C16, C15 to C17, C24 to C18, C25 to C19, C27 to C20, C32 to C21, C28 to C22, C30 to C23, C31 to C24, C39 to C25, C45 to C26, C51 to C27, C41 to C28, C52 to C29, C54 to C30, C58 to C31, C47 to C33, C49 to C34, C50 to C35, C53 to C36, C55 to C37, C56 to C38, C57 to C39, C357 to C40, C59 to C41, C60 to C42, C61 to C43, C359 to C45, C9 to C5, C5 to C6, C6 to C7, C7 to C8, C10 to C9, D10 to D11, D12 to D13, D14 to D15, D16 to D17, D18 to D19, D4 to D5, D6 to D7, D8 to D9, L2 to L1, L3 to L2, L4 to L3, L5 to L4, L6 to L5, L7 to L6, R2 to R1, R13 to R10, R14 to R11, R15 to R12, R16 to R15, R1 to R16, R3 to R2, R6 to R21, R7 to R22, R23 to R25, R25 to R27, R26 to R29, R4 to R3, R28 to R31, R30 to R33, R32 to R35, R34 to R37, R36 to R39, R5 to R4, R38 to R41, R40 to R43, R11 to R8, R12 to R9, TP10 to TP21, TP11 to TP22, TP12 to TP23, TP13 to TP24, TP14 to TP25, TP15 to TP26, TP16 to TP27, TP17 to TP28, U13 to U10, U15 to U11, U17 to U12, U21 to U13, U22 to U14, U6 to U15, U24 to U16, U26 to U17, U27 to U19, U28 to U20, U29 to U21, U30 to U23, U7 to U4, U9 to U5, U5 to U6, U11 to U7, U10 to U9
Connections:
- net GND: now also C32.2, U8.4 (G), U8.5 (G)
- net VDD: now also C32.1
- net VEE: now also U8.3
- net at C14.2, D3.2 (K), U3.22 (VBCOMP)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: now also U8.1
- no-connect marks 25 -> 26
Other:
- note added: "TPS62420 also ok"

Commit message: board nearing completion - at least with routing! seems to be a bug in the netlist, though -- have to check it out.
Parts:
- added C60: 0.1uf, 0402, symbol C
- added R54, R55: 50, 0402, symbol R
- added TP29, TP30: 37, TP, symbol TP
- added TP31: G, TP, symbol TP
Connections:
- net DR0PRI: now also TP5.1
- net DR1PRI: no longer U22.7 (A6)
- net DT0PRI: now also R7.1
- net GND: now also C60.2, TP31.1
- net RFS0: now also TP3.1
- net RSCLK0: now also TP4.1
- net RX: now also R55.1; no longer U2.12 (R1OUT)
- net TFS0: now also R5.1
- net TSCLK0: now also R6.1
- net TX: now also R54.1; no longer U2.11 (T1IN)
- net VCC: now also TP29.1, TP30.1
- net VDD: now also U22.7 (A6), C60.1
- net at R7.2: now also TP10.1; no longer TP5.1
- net at R6.2: now also TP9.1; no longer TP4.1
- net at R5.2: now also TP8.1; no longer TP3.1
- removed net DT1PRI: R7.1, TP10.1, U14.F2 (DT1PRI)
- removed net TFS1: R5.1, TP8.1, U14.E1 (TFS1)
- removed net TSCLK1: R6.1, TP9.1, U14.F1 (TSCLK1)
- new net: R54.2, U2.11 (T1IN)
- new net: R55.2, U2.12 (R1OUT)
Other:
- note added: "for wired headstqage - i guess."
- moved on the sheet: TP1, TP10, TP2, TP3, TP4, TP5, TP8, TP9
