File: emg_dsp/stage6/analog.sch (KiCad schematic (older format))
At the start: 31 parts, among them U75 OMNETICS_36, U76 RHA2116, U77 MIC5365, U78 TC1016, U79 ADCS7476, U80 RHA2116, U81 ADCS7476

Commit message: submitted a (partial) BOM .. !! board is not yet cone, but at least we now know to switch the footprint on the flash.
Parts:
- U77: value MIC5365 -> MIC5365-2.7
- U78: value TC1016 -> TC1016-3.0
Changed lines of the file:
@@
-EESchema Schematic File Version 2  date Thu 30 Sep 2010 05:10:58 PM EDT
+EESchema Schematic File Version 2  date Thu 30 Sep 2010 11:24:56 PM EDT
 LIBS:power
 LIBS:device
@@
 Sheet 13 15
 Title "Stage 4 / Copyright 2010 Timothy L Hanson "
-Date "30 sep 2010"
+Date "1 oct 2010"
 Rev ""
 Comp "This design is free: redistribute or modify under the GPL v. 3 or later"
@@
 P 4500 6000
 F 0 "U77" H 4500 5800 60  0000 C CNN
-F 1 "MIC5365" H 4500 6200 60  0000 C CNN
+F 1 "MIC5365-2.7" H 4500 6200 60  0000 C CNN
 F 2 "SC-70-5" H 4440 5740 60  0000 C CNN
 	1    4500 6000
@@
 $EndComp
 $Comp
-L GND #PWR0376
+L GND #PWR0378
 U 1 1 4C2A3423
 P 8050 650
-F 0 "#PWR0376" H 8050 650 30  0001 C CNN
+F 0 "#PWR0378" H 8050 650 30  0001 C CNN
 F 1 "GND" H 8050 580 30  0001 C CNN
 	1    8050 650
@@
 $EndComp
 $Comp
-L GND #PWR0377
+L GND #PWR0379
 U 1 1 4C2A338B
 P 7300 2850
-F 0 "#PWR0377" H 7300 2850 30  0001 C CNN
+F 0 "#PWR0379" H 7300 2850 30  0001 C CNN
 F 1 "GND" H 7300 2780 30  0001 C CNN
 	1    7300 2850
@@
 $EndComp
 $Comp
-L GND #PWR0378
+L GND #PWR0380
 U 1 1 4C2A338A
 P 8850 3000
-F 0 "#PWR0378" H 8850 3000 30  0001 C CNN
+F 0 "#PWR0380" H 8850 3000 30  0001 C CNN
 F 1 "GND" H 8850 2930 30  0001 C CNN
 	1    8850 3000
@@
 $EndComp
 $Comp
-L GND #PWR0379
+L GND #PWR0381
 U 1 1 4C2A3388
 P 9300 3050
-F 0 "#PWR0379" H 9300 3050 30  0001 C CNN
+F 0 "#PWR0381" H 9300 3050 30  0001 C CNN
 F 1 "GND" H 9300 2980 30  0001 C CNN
 	1    9300 3050
@@
 $EndComp
 $Comp
-L GND #PWR0380
+L GND #PWR0382
 U 1 1 4C2A3386
 P 9100 3900
-F 0 "#PWR0380" H 9100 3900 30  0001 C CNN
+F 0 "#PWR0382" H 9100 3900 30  0001 C CNN
 F 1 "GND" H 9100 3830 30  0001 C CNN
 	1    9100 3900
@@
 $EndComp
 $Comp
-L GND #PWR0381
+L GND #PWR0383
 U 1 1 4C2A3382
 P 9650 1800
-F 0 "#PWR0381" H 9650 1800 30  0001 C CNN
+F 0 "#PWR0383" H 9650 1800 30  0001 C CNN
 F 1 "GND" H 9650 1730 30  0001 C CNN
 	1    9650 1800
@@
 $EndComp
 $Comp
-L GND #PWR0382
+L GND #PWR0384
 U 1 1 4C2A3381
 P 9650 1950
-F 0 "#PWR0382" H 9650 1950 30  0001 C CNN
+F 0 "#PWR0384" H 9650 1950 30  0001 C CNN
 F 1 "GND" H 9650 1880 30  0001 C CNN
 	1    9650 1950
@@
 $EndComp
 $Comp
-L GND #PWR0383
+L GND #PWR0385
 U 1 1 4C2A337F
 P 9650 2100
-F 0 "#PWR0383" H 9650 2100 30  0001 C CNN
+F 0 "#PWR0385" H 9650 2100 30  0001 C CNN
 F 1 "GND" H 9650 2030 30  0001 C CNN
 	1    9650 2100
@@
 $EndComp
 $Comp
-L GND #PWR0384
+L GND #PWR0386
 U 1 1 4C2A337C
 P 8900 1800
-F 0 "#PWR0384" H 8900 1800 30  0001 C CNN
+F 0 "#PWR0386" H 8900 1800 30  0001 C CNN
 F 1 "GND" H 8900 1730 30  0001 C CNN
 	1    8900 1800
@@
 $EndComp
 $Comp
-L GND #PWR0385
+L GND #PWR0387
 U 1 1 4C2A337B
 P 8900 1250
-F 0 "#PWR0385" H 8900 1250 30  0001 C CNN
+F 0 "#PWR0387" H 8900 1250 30  0001 C CNN
 F 1 "GND" H 8900 1180 30  0001 C CNN
 	1    8900 1250
@@
 V3
 $Comp
-L GND #PWR0386
+L GND #PWR0388
 U 1 1 4C2A337A
 P 8900 2350
-F 0 "#PWR0386" H 8900 2350 30  0001 C CNN
+F 0 "#PWR0388" H 8900 2350 30  0001 C CNN
 F 1 "GND" H 8900 2280 30  0001 C CNN
 	1    8900 2350
@@
 $EndComp
 $Comp
-L GND #PWR0387
+L GND #PWR0389
 U 1 1 4C2A3379
 P 8100 3300
-F 0 "#PWR0387" H 8100 3300 30  0001 C CNN
+F 0 "#PWR0389" H 8100 3300 30  0001 C CNN
 F 1 "GND" H 8100 3230 30  0001 C CNN
 	1    8100 3300
@@
 NoConn ~ 3950 3100
 $Comp
-L GND #PWR0388
+L GND #PWR0390
 U 1 1 4C2A32DF
 P 4100 650
-F 0 "#PWR0388" H 4100 650 30  0001 C CNN
+F 0 "#PWR0390" H 4100 650 30  0001 C CNN
 F 1 "GND" H 4100 580 30  0001 C CNN
 	1    4100 650
@@
 $EndComp
 $Comp
-L GND #PWR0389
+L GND #PWR0391
 U 1 1 4C2A32D7
 P 4150 3300
-F 0 "#PWR0389" H 4150 3300 30  0001 C CNN
+F 0 "#PWR0391" H 4150 3300 30  0001 C CNN
 F 1 "GND" H 4150 3230 30  0001 C CNN
 	1    4150 3300
@@
 $EndComp
 $Comp
-L GND #PWR0390
+L GND #PWR0392
 U 1 1 4C2A32BF
 P 4950 2350
-F 0 "#PWR0390" H 4950 2350 30  0001 C CNN
+F 0 "#PWR0392" H 4950 2350 30  0001 C CNN
 F 1 "GND" H 4950 2280 30  0001 C CNN
 	1    4950 2350
@@
 V3
 $Comp
-L GND #PWR0391
+L GND #PWR0393
 U 1 1 4C2A3286
 P 4950 1250
-F 0 "#PWR0391" H 4950 1250 30  0001 C CNN
+F 0 "#PWR0393" H 4950 1250 30  0001 C CNN
 F 1 "GND" H 4950 1180 30  0001 C CNN
 	1    4950 1250
@@
 $EndComp
 $Comp
-L GND #PWR0392
+L GND #PWR0394
 U 1 1 4C2A3267
 P 4950 1800
-F 0 "#PWR0392" H 4950 1800 30  0001 C CNN
+F 0 "#PWR0394" H 4950 1800 30  0001 C CNN
 F 1 "GND" H 4950 1730 30  0001 C CNN
 	1    4950 1800
@@
 $EndComp
 $Comp
-L GND #PWR0393
+L GND #PWR0395
 U 1 1 4C2A3090
 P 5700 2100
-F 0 "#PWR0393" H 5700 2100 30  0001 C CNN
+F 0 "#PWR0395" H 5700 2100 30  0001 C CNN
 F 1 "GND" H 5700 2030 30  0001 C CNN
 	1    5700 2100
@@
 $EndComp
 $Comp
-L GND #PWR0394
+L GND #PWR0396
 U 1 1 4C2A3089
 P 5700 1950
-F 0 "#PWR0394" H 5700 1950 30  0001 C CNN
+F 0 "#PWR0396" H 5700 1950 30  0001 C CNN
 F 1 "GND" H 5700 1880 30  0001 C CNN
 	1    5700 1950
@@
 $EndComp
 $Comp
-L GND #PWR0395
+L GND #PWR0397
 U 1 1 4C2A3084
 P 5700 1800
-F 0 "#PWR0395" H 5700 1800 30  0001 C CNN
+F 0 "#PWR0397" H 5700 1800 30  0001 C CNN
 F 1 "GND" H 5700 1730 30  0001 C CNN
 	1    5700 1800
@@
 V27
 $Comp
-L VDD #PWR0396
+L VDD #PWR0398
 U 1 1 4C2A2EC5
 P 3050 5750
-F 0 "#PWR0396" H 3050 5850 30  0001 C CNN
+F 0 "#PWR0398" H 3050 5850 30  0001 C CNN
 F 1 "VDD" H 3050 5860 30  0000 C CNN
 	1    3050 5750
@@
 $EndComp
 $Comp
-L GND #PWR0397
+L GND #PWR0399
 U 1 1 4C2A2E8B
 P 5150 3900
-F 0 "#PWR0397" H 5150 3900 30  0001 C CNN
+F 0 "#PWR0399" H 5150 3900 30  0001 C CNN
 F 1 "GND" H 5150 3830 30  0001 C CNN
 	1    5150 3900
@@
 $EndComp
 $Comp
-L GND #PWR0398
+L GND #PWR0400
 U 1 1 4C2A2E11
 P 5350 3050
-F 0 "#PWR0398" H 5350 3050 30  0001 C CNN
+F 0 "#PWR0400" H 5350 3050 30  0001 C CNN
 F 1 "GND" H 5350 2980 30  0001 C CNN
 	1    5350 3050
@@
 $EndComp
 $Comp
-L GND #PWR0399
+L GND #PWR0401
 U 1 1 4C2A2DE8
 P 4900 3000
-F 0 "#PWR0399" H 4900 3000 30  0001 C CNN
+F 0 "#PWR0401" H 4900 3000 30  0001 C CNN
 F 1 "GND" H 4900 2930 30  0001 C CNN
 	1    4900 3000
@@
 $EndComp
 $Comp
-L GND #PWR0400
+L GND #PWR0402
 U 1 1 4C2A2DD8
 P 3350 2850
-F 0 "#PWR0400" H 3350 2850 30  0001 C CNN
+F 0 "#PWR0402" H 3350 2850 30  0001 C CNN
 F 1 "GND" H 3350 2780 30  0001 C CNN
 	1    3350 2850
@@
 $EndComp
 $Comp
-L GND #PWR0401
+L GND #PWR0403
 U 1 1 4C2A2B2E
 P 5300 6300
-F 0 "#PWR0401" H 5300 6300 30  0001 C CNN
+F 0 "#PWR0403" H 5300 6300 30  0001 C CNN
 F 1 "GND" H 5300 6230 30  0001 C CNN
 	1    5300 6300
@@
 $EndComp
 $Comp
-L GND #PWR0402
+L GND #PWR0404
 U 1 1 4C2A2B2C
 P 3650 6300
-F 0 "#PWR0402" H 3650 6300 30  0001 C CNN
+F 0 "#PWR0404" H 3650 6300 30  0001 C CNN
 F 1 "GND" H 3650 6230 30  0001 C CNN
 	1    3650 6300
@@
 $EndComp
 $Comp
-L GND #PWR0403
+L GND #PWR0405
 U 1 1 4C2A2B2B
 P 4150 6000
-F 0 "#PWR0403" H 4150 6000 30  0001 C CNN
+F 0 "#PWR0405" H 4150 6000 30  0001 C CNN
 F 1 "GND" H 4150 5930 30  0001 C CNN
 	1    4150 6000
@@
 $EndComp
 $Comp
-L GND #PWR0404
+L GND #PWR0406
 U 1 1 4C2A2B28
 P 3050 6300
-F 0 "#PWR0404" H 3050 6300 30  0001 C CNN
+F 0 "#PWR0406" H 3050 6300 30  0001 C CNN
 F 1 "GND" H 3050 6230 30  0001 C CNN
 	1    3050 6300
@@
 P 4750 4950
 F 0 "U78" H 4750 4750 60  0000 C CNN
-F 1 "TC1016" H 4750 5150 60  0000 C CNN
+F 1 "TC1016-3.0" H 4750 5150 60  0000 C CNN
 F 2 "SC-70-5" H 4700 4650 60  0000 C CNN
 	1    4750 4950
@@
 $EndComp
 $Comp
-L VEE #PWR328
+L VEE #PWR329
 U 1 1 4C2A12C9
 P 3050 4500
-F 0 "#PWR328" H 3050 4700 40  0001 C CNN
+F 0 "#PWR329" H 3050 4700 40  0001 C CNN
 F 1 "VEE" H 3050 4650 40  0000 C CNN
 	1    3050 4500
@@
 $EndComp
 $Comp
-L GND #PWR0405
+L GND #PWR0407
 U 1 1 4B69FA06
 P 3050 5050
-F 0 "#PWR0405" H 3050 5050 30  0001 C CNN
+F 0 "#PWR0407" H 3050 5050 30  0001 C CNN
 F 1 "GND" H 3050 4980 30  0001 C CNN
 	1    3050 5050
@@
 $EndComp
 $Comp
-L GND #PWR0406
+L GND #PWR0408
 U 1 1 4CA0ED5B
 P 1550 3100
-F 0 "#PWR0406" H 1550 3100 30  0001 C CNN
+F 0 "#PWR0408" H 1550 3100 30  0001 C CNN
 F 1 "GND" H 1550 3030 30  0001 C CNN
 	1    1550 3100
@@
 $EndComp
 $Comp
-L GND #PWR0407
+L GND #PWR0409
 U 1 1 4CA0ED5A
 P 1550 700
-F 0 "#PWR0407" H 1550 700 30  0001 C CNN
+F 0 "#PWR0409" H 1550 700 30  0001 C CNN
 F 1 "GND" H 1550 630 30  0001 C CNN
 	1    1550 700
@@
 V3
 $Comp
-L GND #PWR0408
+L GND #PWR0410
 U 1 1 48FFF0EE
 P 4850 5400
-F 0 "#PWR0408" H 4850 5400 30  0001 C CNN
+F 0 "#PWR0410" H 4850 5400 30  0001 C CNN
 F 1 "GND" H 4850 5330 30  0001 C CNN
 	1    4850 5400
@@
 $EndComp
 $Comp
-L GND #PWR0409
+L GND #PWR0411
 U 1 1 48FFF0D4
 P 3900 5050
-F 0 "#PWR0409" H 3900 5050 30  0001 C CNN
+F 0 "#PWR0411" H 3900 5050 30  0001 C CNN
 F 1 "GND" H 3900 4980 30  0001 C CNN
 	1    3900 5050
@@
 $EndComp
 $Comp
-L GND #PWR0410
+L GND #PWR0412
 U 1 1 48FFF041
 P 5300 5050
-F 0 "#PWR0410" H 5300 5050 30  0001 C CNN
+F 0 "#PWR0412" H 5300 5050 30  0001 C CNN
 F 1 "GND" H 5300 4980 30  0001 C CNN
 	1    5300 5050
