File: emg_dsp/stage6/emg.sch (KiCad schematic (older format))
At the start: 149 parts, among them U53 8X2X100, U54 VEE, U55 MIC5365, U56 AD7689, U57 GT12MABE, U58 LM828, U59 MIC5365, U60 74LVC1G, U61 TPS62410, U62 EN_VCC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

Commit message: getting closer -- needt o put DACs on the board so we can listen to the emg / neural data!
Parts:
- added C?: 0.1uf, 0402, symbol C
Connections:
- net GND: now also C?.1
- net at C116.1, U56.1 (VDD), U56.15 (VIO)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: now also C?.2
Changed lines of the file:
@@
-EESchema Schematic File Version 2  date Wed 29 Sep 2010 05:47:59 PM EDT
+EESchema Schematic File Version 2  date Thu 30 Sep 2010 12:31:09 AM EDT
 LIBS:power
 LIBS:device
@@
 Sheet 2 13
 Title "Stage 4 / Copyright 2010 Timothy L Hanson "
-Date "29 sep 2010"
+Date "30 sep 2010"
 Rev ""
 Comp "This design is free: redistribute or modify under the GPL v. 3 or later"
@@
 Comment4 ""
 $EndDescr
+$Comp
+L GND #PWR?
+U 1 1 4CA41285
+P 3550 2350
+F 0 "#PWR?" H 3550 2350 30  0001 C CNN
+F 1 "GND" H 3550 2280 30  0001 C CNN
+	1    3550 2350
+	0    -1   -1   0
+$EndComp
+$Comp
+L C C?
+U 1 1 4CA4127C
+P 3350 2350
+F 0 "C?" H 3400 2450 50  0000 L CNN
+F 1 "0.1uf" H 3400 2250 50  0000 L CNN
+F 2 "0402" H 3450 2500 60  0000 C CNN
+	1    3350 2350
+	0    1    1    0
+$EndComp
 Connection ~ 8250 750
 Wire Wire Line

Commit message: added audio out to both the wireless-emg and bridge -- very simple circut, sholud work.  layout maybe 70% done.
Parts:
- added R192, R193, R194: 33, 0402, symbol R
- C111: footprint 2x100mil -> 2917
- gave numbers to parts that had none: 1
Connections:
- net at U65.E1 (TFS1): now also R193.1
- net at U65.F1 (TSCLK1): now also R194.1
- net at U65.F2 (DT1PRI): now also R192.1
- new net DT1PRI: R192.2
- new net TFS1: R193.2
- new net TSCLK1: R194.2
- no-connect marks 10 -> 7
Other:
- moved on the sheet: R107, R113, R114, U66

Commit message: submitted a (partial) BOM .. !! board is not yet cone, but at least we now know to switch the footprint on the flash.
Parts:
- U55, U59: value MIC5365 -> MIC5365-2.7
- U64: value ABM10XTAL -> ABM10XTAL-16
- U69: footprint UFDN-8 -> SOIC-8

Commit message: getting the last of the nets (GND, Vdd, Vcc) routed. still need to check the pinouts, etc.
Parts:
- added C249, C250, C251, C252: 2.2uf, 0402, symbol C
- added C253, C254, C255: 0.1uf, 0402, symbol C
Connections:
- net GND: now also C249.2, C250.2, C251.2, C252.2, C253.2, C254.2, C255.2
- net VDD: now also C253.1, C254.1, C255.1
- net VEMG+: now also C250.1, C251.1
- net VEMG-: now also C249.1, C252.1

Commit message: board getting done! next up is silkscreen - pita.
Parts:
- added TP68, TP69, TP70, TP71: TP, 2.9mm_hole, symbol TP
Connections:
- net GND: now also TP68.1, TP69.1, TP70.1, TP71.1
