File: emg_dsp/stage6/neuro.sch (KiCad schematic (older format))
At the start: 92 parts, among them U24 VEE, U25 74LCX541, U26 TPS62410, U27 EN_VCC, U28 EN_VDD, U29 ABM10XTAL, U30 BF532-160, U31 ADSP_JTAG_CON, U32 NRF24L01, U33 AT25DF041-MHF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

Commit message: neuro part mostly layed out ...
Parts:
- removed U27: EN_VCC, 2x100mil, symbol JUMP
- removed U28: EN_VDD, 2x100mil, symbol JUMP
Connections:
- net VCC: no longer TP28.1
- net VDD: no longer TP26.1
- net VEE: no longer TP30.1
- net at C53.2, C54.2, C55.2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: now also TP30.1
- net at C63.2, L6.2, R64.1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: now also TP26.1
- net at C61.1, C62.2, L5.2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: now also TP28.1
Other:
- moved on the sheet: TP26, TP28, TP30

Commit message: ethernet partially routed, SDRAM mostly / completely routed. getting there!
Connections:
- net GND: now also U24.1
- net VEE: no longer U24.1

Commit message: submitted a (partial) BOM .. !! board is not yet cone, but at least we now know to switch the footprint on the flash.
Parts:
- U29: value ABM10XTAL -> ABM10XTAL-16
- U33: footprint UFDN-8 -> SOIC-8
