File: emg_dsp/stage8/analog.sch (KiCad schematic (older format))
At the start: 22 parts, among them U75 OMNETICS_36, U77 MIC5365-2.8, U78 TC1016-3.0

Commit message: another damn board! well, at least it's going faster. (not too much changed)
Parts:
- removed R?: 0, 0402, symbol R
- removed U?: RHA2132, symbol RHA2132
- added R67, R70: 0, 0201, symbol R
- added R71, R72, R76, R78: 200, 0402, symbol R
- added U45: RHA2132, QFN-56, symbol RHA2132
- R68, R69: renamed from R?; footprint 0402 -> 0201
- U36: renamed from U77; value MIC5365-2.8 -> MIC5365-2.7
- gave numbers to parts that had none: 11
- renumbered C153 to C59, C154 to C60, C158 to C61, C159 to C62, U75 to U35, U78 to U37
Connections:
- net CS: now also R76.1; no longer U39.6, U40.6 (_cs), U41.6
- net DATA: now also U41.7; no longer U41.3
- net E1: now also U35.2 (in1), U45.34 (in31); no longer U35.17 (in16)
- net E10: now also U35.11 (in10), U45.43 (in22); no longer U35.8 (in7)
- net E11: now also U35.12 (in11), U45.44 (in21); no longer U35.7 (in6)
- net E12: now also U35.13 (in12), U45.45 (in20); no longer U35.6 (in5)
- net E13: now also U35.14 (in13), U45.46 (in19); no longer U35.5 (in4)
- net E14: now also U35.15 (in14), U45.47 (in18); no longer U35.4 (in3)
- net E15: now also U35.16 (in15), U45.48 (in17); no longer U35.3 (in2)
- net E16: now also U35.17 (in16), U45.49 (in16); no longer U35.2 (in1)
- net E17: now also U45.50 (in15)
- net E18: now also U45.51 (in14)
- net E19: now also U45.52 (in13)
- net E2: now also U35.3 (in2), U45.35 (in30); no longer U35.16 (in15)
- net E20: now also U45.53 (in12)
- net E21: now also U45.54 (in11)
- net E22: now also U45.55 (in10)
- net E23: now also U45.56 (in9)
- net E24: now also U45.1 (in8)
- net E25: now also U45.2 (in7)
- net E26: now also U45.3 (in6)
- net E27: now also U45.4 (in5)
- net E28: now also U45.5 (in4)
- net E29: now also U45.6 (in3)
- net E3: now also U35.4 (in3), U45.36 (in29); no longer U35.15 (in14)
- net E30: now also U45.7 (in2)
- net E31: now also U45.8 (in1)
- net E32: now also U45.9 (in0)
- net E4: now also U35.5 (in4), U45.37 (in28); no longer U35.14 (in13)
- net E5: now also U35.6 (in5), U45.38 (in27); no longer U35.13 (in12)
- net E6: now also U35.7 (in6), U45.39 (in26); no longer U35.12 (in11)
- net E7: now also U35.8 (in7), U45.40 (in25); no longer U35.11 (in10)
- net E8: now also U35.9 (in8), U45.41 (in24); no longer U35.10 (in9)
- net E9: now also U35.10 (in9), U45.42 (in23); no longer U35.9 (in8)
- net GND: now also U45.11 (AGND), U45.13 (AGND), U45.19 (settle), U45.28 (DGND), U45.29 (DGND), U45.30 (test_en), U45.31 (conn_all), U45.32 (VESD), U45.33 (elec_test), U45.57 (PAD)
- net RESET: now also R71.1; no longer U39.7, U41.7
- net SCLK: now also R78.1; no longer U39.4, U40.4 (Sclk), U41.4
- net STEP: now also R72.1; no longer U39.9, U41.9
- net V3: now also U45.12 (AVDD), U45.25 (Mode), U45.27 (DVDD)
- net VEE: now also U41.9; no longer U41.1
- net at R68.2, U35.1 (Ref2): now also R67.1
- net at R69.1, U35.36 (Ref1): now also R70.2
- net at R73.2: now also U45.14 (setH1)
- net at R74.2: now also U45.15 (setH2)
- net at R75.2: now also U45.16 (setL)
- net at U40.3 (Vin): now also U45.18 (MUX_out)
- new net: R67.2, R70.1, U45.10 (ref_elec)
- new net Sclk-l: R78.2, U39.4, U40.4 (Sclk), U41.6
- new net _cs: R76.2, U39.6, U40.6 (_cs), U41.4
- new net reset-l: R71.2, U39.7, U41.3, U45.20 (~reset)
- new net step-l: R72.2, U39.9, U41.1, U45.21 (step)
