File: emg_dsp/stage8/stage8.sch (KiCad schematic (older format))
At the start: 101 parts, among them U1 VEE, U10 74LCX541, U11 MAX6711Z, U12 ANTENNA, U13 TESTCON, U2 74LCX541, U3 9X100, U4 TPS62410, U5 ABM10XTAL-16, U6 BF532-160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

Commit message: laaayout!
Connections:
- net RSCLK1 is gone; now on net RSCLK0: U6.G1 (RSCLK1)
- net DR0SEC: no longer U6.F3 (DR1SEC)
- new net DR1SEC: U6.F3 (DR1SEC)

Commit message: layout basically done -- need the routing outline.
Connections:
- net VCC: now also C13.2, L2.2, R15.1, TP10.1, U4.4 (FB1)
- net VDD: now also C11.1, C12.2, L1.2, R14.2, TP9.1
- net Vbat renamed VEE
