File: emg_dsp/stage8/stage8.sch (KiCad schematic (older format))
At the start: 101 parts, among them U1 VEE, U10 74LCX541, U11 MAX6711Z, U12 ANTENNA, U13 TESTCON, U2 74LCX541, U3 9X100, U4 TPS62410, U5 ABM10XTAL-16, U6 BF532-160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

Commit message: spreadsheet for the robot.
Other:
- note added: "to get 0.95v: \n160/270k or 115/195k"
Changed lines of the file:
@@
-EESchema Schematic File Version 2  date Thu 20 Jan 2011 11:51:19 AM EST
+EESchema Schematic File Version 2  date Tue 01 Nov 2011 04:41:02 PM EDT
 LIBS:power
 LIBS:device
@@
 Sheet 1 5
 Title "Stage 4 / Copyright 2010 Timothy L Hanson "
-Date "20 jan 2011"
+Date "1 nov 2011"
 Rev ""
 Comp "This design is free: redistribute or modify under the GPL v. 3 or later"
@@
 Comment4 ""
 $EndDescr
+Text Notes 7000 9450 0    60   ~ 0
+to get 0.95v: \n160/270k or 115/195k
 Wire Wire Line
 	3650 8050 3650 8650
