File: emg_dsp/stage7/wired.sch (KiCad schematic (older format))
At the start: 20 parts, among them U43 9X100, U44 LT1721, U45 TC1016-3.0, U46 DCP01DB, U47 IL715-3

Commit message: layout - stage 7 - got SDRAM and part of the Eth phy routed well. getting the rest of the components in their approx end positions.
Parts:
- added C146: 0.1uf, 0402, symbol C
Connections:
- net V0b: now also C146.1
- net V3C: now also C146.2
Changed lines of the file:
@@
-EESchema Schematic File Version 2  date Wed 26 Jan 2011 02:24:37 PM EST
+EESchema Schematic File Version 2  date Thu 27 Jan 2011 02:09:10 PM EST
 LIBS:power
 LIBS:device
@@
 Sheet 2 19
 Title "Stage 4 / Copyright 2010 Timothy L Hanson "
-Date "26 jan 2011"
+Date "27 jan 2011"
 Rev ""
 Comp "This design is free: redistribute or modify under the GPL v. 3 or later"
@@
 Comment4 ""
 $EndDescr
+Connection ~ 12100 3150
+Wire Wire Line
+	12500 2800 12500 3150
+Wire Wire Line
+	12500 3150 9600 3150
 Connection ~ 7700 4800
 Wire Wire Line
@@
 Connection ~ 11600 3150
 Wire Wire Line
-	12100 2800 12100 3150
-Wire Wire Line
-	12100 3150 9600 3150
+	12100 3150 12100 2800
 Connection ~ 11650 5700
 Wire Wire Line
@@
 	11450 5300 12150 5300
 Connection ~ 11650 5300
-Wire Wire Line
-	12100 2400 10550 2400
 Connection ~ 11600 2400
 Wire Wire Line
@@
 	7700 4200 7700 4300
 Connection ~ 8050 4200
+Wire Wire Line
+	12500 2400 10550 2400
+Connection ~ 12100 2400
+$Comp
+L C C146
+U 1 1 4D41AD4D
+P 12500 2600
+F 0 "C146" H 12550 2700 50  0000 L CNN
+F 1 "0.1uf" H 12550 2500 50  0000 L CNN
+F 2 "0402" H 12600 2750 60  0000 C CNN
+	1    12500 2600
+	-1   0    0    1
+$EndComp
 $Comp
 L C C92
@@
 $EndComp
 $Comp
-L VEE #PWR203
+L VEE #PWR195
 U 1 1 4C9B878C
 P 11250 5450
-F 0 "#PWR203" H 11250 5650 40  0001 C CNN
+F 0 "#PWR195" H 11250 5650 40  0001 C CNN
 F 1 "VEE" H 11250 5600 40  0000 C CNN
 	1    11250 5450

Commit message: getting there! about 70-80% done with individual routing.
Parts:
- added C?: 0.1uf, 0402, symbol C
Connections:
- net GND: now also C?.1
- net VDD: now also C?.2
Changed lines of the file:
@@
-EESchema Schematic File Version 2  date Thu 27 Jan 2011 02:09:10 PM EST
+EESchema Schematic File Version 2  date Thu 27 Jan 2011 05:22:18 PM EST
 LIBS:power
 LIBS:device
@@
 Comment4 ""
 $EndDescr
+$Comp
+L VDD #PWR?
+U 1 1 4D41F018
+P 13150 3550
+F 0 "#PWR?" H 13150 3650 30  0001 C CNN
+F 1 "VDD" H 13150 3660 30  0000 C CNN
+	1    13150 3550
+	1    0    0    -1
+$EndComp
+$Comp
+L GND #PWR?
+U 1 1 4D41F014
+P 13150 3950
+F 0 "#PWR?" H 13150 3950 30  0001 C CNN
+F 1 "GND" H 13150 3880 30  0001 C CNN
+	1    13150 3950
+	1    0    0    -1
+$EndComp
+$Comp
+L C C?
+U 1 1 4D41F00F
+P 13150 3750
+F 0 "C?" H 13200 3850 50  0000 L CNN
+F 1 "0.1uf" H 13200 3650 50  0000 L CNN
+F 2 "0402" H 13250 3900 60  0000 C CNN
+	1    13150 3750
+	-1   0    0    1
+$EndComp
 Connection ~ 12100 3150
 Wire Wire Line
@@
 NoConn ~ 11250 5750
 $Comp
-L GND #PWR0139
+L GND #PWR0136
 U 1 1 4C9B9212
 P 12350 4150
-F 0 "#PWR0139" H 12350 4150 30  0001 C CNN
+F 0 "#PWR0136" H 12350 4150 30  0001 C CNN
 F 1 "GND" H 12350 4080 30  0001 C CNN
 	1    12350 4150
@@
 $EndComp
 $Comp
-L GND #PWR0140
+L GND #PWR0137
 U 1 1 4C9B920A
 P 12350 3550
-F 0 "#PWR0140" H 12350 3550 30  0001 C CNN
+F 0 "#PWR0137" H 12350 3550 30  0001 C CNN
 F 1 "GND" H 12350 3480 30  0001 C CNN
 	1    12350 3550
@@
 $EndComp
 $Comp
-L VDD #PWR0141
+L VDD #PWR0138
 U 1 1 4C9B9204
 P 12300 3450
-F 0 "#PWR0141" H 12300 3550 30  0001 C CNN
+F 0 "#PWR0138" H 12300 3550 30  0001 C CNN
 F 1 "VDD" H 12300 3560 30  0000 C CNN
 	1    12300 3450
@@
 $EndComp
 $Comp
-L GND #PWR0142
+L GND #PWR0139
 U 1 1 4C9B8790
 P 11300 5600
-F 0 "#PWR0142" H 11300 5600 30  0001 C CNN
+F 0 "#PWR0139" H 11300 5600 30  0001 C CNN
 F 1 "GND" H 11300 5530 30  0001 C CNN
 	1    11300 5600
@@
 $EndComp
 $Comp
-L VEE #PWR195
+L VEE #PWR192
 U 1 1 4C9B878C
 P 11250 5450
-F 0 "#PWR195" H 11250 5650 40  0001 C CNN
+F 0 "#PWR192" H 11250 5650 40  0001 C CNN
 F 1 "VEE" H 11250 5600 40  0000 C CNN
 	1    11250 5450

Commit message: layout of stage7 just about finished! need to check and make gerbers..
Parts:
- gave numbers to parts that had none: 1
Connections:
- net V3b is gone; now on net V3C: R87.2
Changed lines of the file:
@@
-EESchema Schematic File Version 2  date Thu 27 Jan 2011 05:22:18 PM EST
+EESchema Schematic File Version 2  date Mon 31 Jan 2011 04:09:41 PM EST
 LIBS:power
 LIBS:device
@@
 Sheet 2 19
 Title "Stage 4 / Copyright 2010 Timothy L Hanson "
-Date "27 jan 2011"
+Date "31 jan 2011"
 Rev ""
 Comp "This design is free: redistribute or modify under the GPL v. 3 or later"
@@
 $EndDescr
 $Comp
-L VDD #PWR?
+L VDD #PWR0137
 U 1 1 4D41F018
 P 13150 3550
-F 0 "#PWR?" H 13150 3650 30  0001 C CNN
+F 0 "#PWR0137" H 13150 3650 30  0001 C CNN
 F 1 "VDD" H 13150 3660 30  0000 C CNN
 	1    13150 3550
@@
 $EndComp
 $Comp
-L GND #PWR?
+L GND #PWR0138
 U 1 1 4D41F014
 P 13150 3950
-F 0 "#PWR?" H 13150 3950 30  0001 C CNN
+F 0 "#PWR0138" H 13150 3950 30  0001 C CNN
 F 1 "GND" H 13150 3880 30  0001 C CNN
 	1    13150 3950
@@
 $EndComp
 $Comp
-L C C?
+L C C147
 U 1 1 4D41F00F
 P 13150 3750
-F 0 "C?" H 13200 3850 50  0000 L CNN
+F 0 "C147" H 13200 3850 50  0000 L CNN
 F 1 "0.1uf" H 13200 3650 50  0000 L CNN
 F 2 "0402" H 13250 3900 60  0000 C CNN
@@
 $EndComp
 Text Label 8350 2750 0    60   ~ 0
-V3b
+V3C
 $Comp
 L R R87
@@
 NoConn ~ 11250 5750
 $Comp
-L GND #PWR0136
+L GND #PWR0139
 U 1 1 4C9B9212
 P 12350 4150
-F 0 "#PWR0136" H 12350 4150 30  0001 C CNN
+F 0 "#PWR0139" H 12350 4150 30  0001 C CNN
 F 1 "GND" H 12350 4080 30  0001 C CNN
 	1    12350 4150
@@
 $EndComp
 $Comp
-L GND #PWR0137
+L GND #PWR0140
 U 1 1 4C9B920A
 P 12350 3550
-F 0 "#PWR0137" H 12350 3550 30  0001 C CNN
+F 0 "#PWR0140" H 12350 3550 30  0001 C CNN
 F 1 "GND" H 12350 3480 30  0001 C CNN
 	1    12350 3550
@@
 $EndComp
 $Comp
-L VDD #PWR0138
+L VDD #PWR0141
 U 1 1 4C9B9204
 P 12300 3450
-F 0 "#PWR0138" H 12300 3550 30  0001 C CNN
+F 0 "#PWR0141" H 12300 3550 30  0001 C CNN
 F 1 "VDD" H 12300 3560 30  0000 C CNN
 	1    12300 3450
@@
 $EndComp
 $Comp
-L GND #PWR0139
+L GND #PWR0142
 U 1 1 4C9B8790
 P 11300 5600
-F 0 "#PWR0139" H 11300 5600 30  0001 C CNN
+F 0 "#PWR0142" H 11300 5600 30  0001 C CNN
 F 1 "GND" H 11300 5530 30  0001 C CNN
 	1    11300 5600
@@
 $EndComp
 $Comp
-L VEE #PWR192
+L VEE #PWR185
 U 1 1 4C9B878C
 P 11250 5450
-F 0 "#PWR192" H 11250 5650 40  0001 C CNN
+F 0 "#PWR185" H 11250 5650 40  0001 C CNN
 F 1 "VEE" H 11250 5600 40  0000 C CNN
 	1    11250 5450
