File: emg_dsp/stage10/audioout.sch (KiCad schematic (older format))
At the start: 17 parts, among them U27 MIC5365-2.5, U28 AD5663, U29 LM4808, U30 AUDIO_JACK

Commit message: word, schematics for 9/10 are close to done. start changing the boards...
Parts:
- C70, C71: value 200uf -> 150uf
Changed lines of the file:
@@
-EESchema Schematic File Version 2  date Tue 11 Oct 2011 02:19:03 AM EDT
+EESchema Schematic File Version 2  date Tue 11 Oct 2011 04:24:56 PM EDT
 LIBS:power
 LIBS:device
@@
 EELAYER END
 $Descr A4 11700 8267
-Sheet 20 3
+Sheet 3 3
 Title ""
 Date "11 oct 2011"
@@
 $EndDescr
 $Comp
-L VDD #PWR0161
+L VDD #PWR0175
 U 1 1 4CACDD2B
 P 6100 3000
-F 0 "#PWR0161" H 6100 3100 30  0001 C CNN
+F 0 "#PWR0175" H 6100 3100 30  0001 C CNN
 F 1 "VDD" H 6100 3110 30  0000 C CNN
 	1    6100 3000
@@
 $EndComp
 $Comp
-L VDD #PWR0162
+L VDD #PWR0176
 U 1 1 4CACDD1E
 P 1700 2350
-F 0 "#PWR0162" H 1700 2450 30  0001 C CNN
+F 0 "#PWR0176" H 1700 2450 30  0001 C CNN
 F 1 "VDD" H 1700 2460 30  0000 C CNN
 	1    1700 2350
@@
 	6950 2950 6950 2850
 $Comp
-L GND #PWR0163
+L GND #PWR0177
 U 1 1 4CA4FCDF
 P 1300 2550
-F 0 "#PWR0163" H 1300 2550 30  0001 C CNN
+F 0 "#PWR0177" H 1300 2550 30  0001 C CNN
 F 1 "GND" H 1300 2480 30  0001 C CNN
 	1    1300 2550
@@
 $EndComp
 $Comp
-L GND #PWR0164
+L GND #PWR0178
 U 1 1 4CA4E84E
 P 6950 3900
-F 0 "#PWR0164" H 6950 3900 30  0001 C CNN
+F 0 "#PWR0178" H 6950 3900 30  0001 C CNN
 F 1 "GND" H 6950 3830 30  0001 C CNN
 	1    6950 3900
@@
 $EndComp
 $Comp
-L GND #PWR0165
+L GND #PWR0179
 U 1 1 4CA4E84C
 P 6950 2350
-F 0 "#PWR0165" H 6950 2350 30  0001 C CNN
+F 0 "#PWR0179" H 6950 2350 30  0001 C CNN
 F 1 "GND" H 6950 2280 30  0001 C CNN
 	1    6950 2350
@@
 $EndComp
 $Comp
-L GND #PWR0166
+L GND #PWR0180
 U 1 1 4CA4E7B7
 P 2650 2750
-F 0 "#PWR0166" H 2650 2750 30  0001 C CNN
+F 0 "#PWR0180" H 2650 2750 30  0001 C CNN
 F 1 "GND" H 2650 2680 30  0001 C CNN
 	1    2650 2750
@@
 $EndComp
 $Comp
-L GND #PWR0167
+L GND #PWR0181
 U 1 1 4CA4E788
 P 1850 2450
-F 0 "#PWR0167" H 1850 2450 30  0001 C CNN
+F 0 "#PWR0181" H 1850 2450 30  0001 C CNN
 F 1 "GND" H 1850 2380 30  0001 C CNN
 	1    1850 2450
@@
 P 6750 3300
 F 0 "C71" H 6800 3400 50  0000 L CNN
-F 1 "200uf" H 6800 3200 50  0000 L CNN
+F 1 "150uf" H 6800 3200 50  0000 L CNN
 F 2 "2917" H 6850 3450 60  0000 C CNN
 	1    6750 3300
@@
 $EndComp
 $Comp
-L GND #PWR0168
+L GND #PWR0182
 U 1 1 4CA4E6A8
 P 7200 3700
-F 0 "#PWR0168" H 7200 3700 30  0001 C CNN
+F 0 "#PWR0182" H 7200 3700 30  0001 C CNN
 F 1 "GND" H 7200 3630 30  0001 C CNN
 	1    7200 3700
@@
 P 6750 2950
 F 0 "C70" H 6800 3050 50  0000 L CNN
-F 1 "200uf" H 6800 2850 50  0000 L CNN
+F 1 "150uf" H 6800 2850 50  0000 L CNN
 F 2 "2917" H 6850 3100 60  0000 C CNN
 	1    6750 2950
@@
 $EndComp
 $Comp
-L GND #PWR0169
+L GND #PWR0183
 U 1 1 4CA4E652
 P 5000 3300
-F 0 "#PWR0169" H 5000 3300 30  0001 C CNN
+F 0 "#PWR0183" H 5000 3300 30  0001 C CNN
 F 1 "GND" H 5000 3230 30  0001 C CNN
 	1    5000 3300
@@
 Vin+
 $Comp
-L GND #PWR0170
+L GND #PWR0184
 U 1 1 4CA4E5F5
 P 4000 3300
-F 0 "#PWR0170" H 4000 3300 30  0001 C CNN
+F 0 "#PWR0184" H 4000 3300 30  0001 C CNN
 F 1 "GND" H 4000 3230 30  0001 C CNN
 	1    4000 3300
@@
 $EndComp
 $Comp
-L GND #PWR0171
+L GND #PWR0185
 U 1 1 4CA4E5B2
 P 4500 2550
-F 0 "#PWR0171" H 4500 2550 30  0001 C CNN
+F 0 "#PWR0185" H 4500 2550 30  0001 C CNN
 F 1 "GND" H 4500 2480 30  0001 C CNN
 	1    4500 2550
@@
 $EndComp
 $Comp
-L GND #PWR0172
+L GND #PWR0186
 U 1 1 4CA4E5AA
 P 4500 3550
-F 0 "#PWR0172" H 4500 3550 30  0001 C CNN
+F 0 "#PWR0186" H 4500 3550 30  0001 C CNN
 F 1 "GND" H 4500 3480 30  0001 C CNN
 	1    4500 3550
@@
 $EndComp
 $Comp
-L GND #PWR0173
+L GND #PWR0187
 U 1 1 4CA4E599
 P 4500 3550
-F 0 "#PWR0173" H 4500 3550 30  0001 C CNN
+F 0 "#PWR0187" H 4500 3550 30  0001 C CNN
 F 1 "GND" H 4500 3480 30  0001 C CNN
 	1    4500 3550
@@
 $EndComp
 $Comp
-L GND #PWR0174
+L GND #PWR0188
 U 1 1 4CA4E4BA
 P 6100 3450
-F 0 "#PWR0174" H 6100 3450 30  0001 C CNN
+F 0 "#PWR0188" H 6100 3450 30  0001 C CNN
 F 1 "GND" H 6100 3380 30  0001 C CNN
 	1    6100 3450
@@
 Vin+
 $Comp
-L GND #PWR0175
+L GND #PWR0189
 U 1 1 4CA4E458
 P 2150 3550
-F 0 "#PWR0175" H 2150 3550 30  0001 C CNN
+F 0 "#PWR0189" H 2150 3550 30  0001 C CNN
 F 1 "GND" H 2150 3480 30  0001 C CNN
 	1    2150 3550
@@
 $EndComp
 $Comp
-L GND #PWR0176
+L GND #PWR0190
 U 1 1 4CA4E455
 P 1700 3550
-F 0 "#PWR0176" H 1700 3550 30  0001 C CNN
+F 0 "#PWR0190" H 1700 3550 30  0001 C CNN
 F 1 "GND" H 1700 3480 30  0001 C CNN
 	1    1700 3550
