File: emg_dsp/stage10/poe.sch (KiCad schematic (older format))
At the start: 40 parts

Commit message: word, schematics for 9/10 are close to done. start changing the boards...
Parts:
- R124: renamed from R?; footprint (none) -> 0402
- U38: renamed from U?; footprint (none) -> SOT-23-6
- U39: renamed from U?; footprint (none) -> DIP-4
- U40: renamed from U?; footprint (none) -> POE13W
- U41: renamed from U?; footprint (none) -> SOT-23
- gave numbers to parts that had none: 35
Other:
- note added: "493-1665-ND"

Commit message: working on board layout for stage10 .. time for the checks!
Parts:
- removed C79: 63uf, 2x200mil, symbol C
- added C92: 63uf, 2x200mil, symbol C
- added C93: 4.7uf, 1210, symbol C
Connections:
- net GND: now also U40.10, U40.11, U40.12
- net GNDPWR: now also C92.2, C93.2
- net POE+: now also C92.1, C93.1
Changed lines of the file:
@@
-EESchema Schematic File Version 2  date Tue 11 Oct 2011 04:24:56 PM EDT
+EESchema Schematic File Version 2  date Wed 12 Oct 2011 06:08:50 PM EDT
 LIBS:power
 LIBS:device
@@
 Sheet 2 3
 Title ""
-Date "11 oct 2011"
+Date "12 oct 2011"
 Rev ""
 Comp ""
@@
 Comment4 ""
 $EndDescr
-Text Notes 3400 2300 0    60   ~ 0
-493-1665-ND
+Connection ~ 2700 1550
+Wire Wire Line
+	2700 1650 2700 1550
 Wire Wire Line
 	9150 2050 8050 2050
@@
 	7450 2350 7250 2350
 Wire Wire Line
-	7250 2550 7350 2550
-Wire Wire Line
-	7350 2550 7350 1950
-Wire Wire Line
-	7350 1950 7250 1950
+	7350 2550 7250 2550
+Wire Wire Line
+	7250 1950 7350 1950
 Wire Wire Line
 	6300 3400 6300 3500
@@
 Wire Wire Line
 	6300 3500 6700 3500
+Wire Wire Line
+	7350 1950 7350 2600
+Connection ~ 7350 2550
+$Comp
+L C C93
+U 1 1 4E95D94F
+P 3600 1850
+F 0 "C93" H 3650 1950 50  0000 L CNN
+F 1 "4.7uf" H 3800 1950 50  0000 L CNN
+F 2 "1210" H 3700 2000 60  0000 C CNN
+	1    3600 1850
+	1    0    0    -1
+$EndComp
+$Comp
+L C C92
+U 1 1 4E95D94B
+P 2700 1850
+F 0 "C92" H 2750 1950 50  0000 L CNN
+F 1 "63uf" H 2900 1950 50  0000 L CNN
+F 2 "2x200mil" H 2950 1850 60  0000 C CNN
+	1    2700 1850
+	1    0    0    -1
+$EndComp
+$Comp
+L GNDPWR #PWR0163
+U 1 1 4E95D94A
+P 2700 2050
+F 0 "#PWR0163" H 2700 2100 40  0001 C CNN
+F 1 "GNDPWR" H 2700 1970 40  0000 C CNN
+	1    2700 2050
+	1    0    0    -1
+$EndComp
+Text Notes 2500 2300 0    60   ~ 0
+493-1665-ND
+$Comp
+L GND #PWR0164
+U 1 1 4E95CAD6
+P 7350 2600
+F 0 "#PWR0164" H 7350 2600 30  0001 C CNN
+F 1 "GND" H 7350 2530 30  0001 C CNN
+	1    7350 2600
+	1    0    0    -1
+$EndComp
+Text Notes 3400 2300 0    60   ~ 0
+493-1665-ND
 $Comp
 L C C80
@@
 $EndComp
 $Comp
-L GNDPWR #PWR0162
+L GNDPWR #PWR0165
 U 1 1 4E93CF88
 P 6700 3900
-F 0 "#PWR0162" H 6700 3950 40  0001 C CNN
+F 0 "#PWR0165" H 6700 3950 40  0001 C CNN
 F 1 "GNDPWR" H 6700 3820 40  0000 C CNN
 	1    6700 3900
@@
 $EndComp
 $Comp
-L GNDPWR #PWR0163
+L GNDPWR #PWR0166
 U 1 1 4E93CEC7
 P 3600 2050
-F 0 "#PWR0163" H 3600 2100 40  0001 C CNN
+F 0 "#PWR0166" H 3600 2100 40  0001 C CNN
 F 1 "GNDPWR" H 3600 1970 40  0000 C CNN
 	1    3600 2050
@@
 $EndComp
 $Comp
-L GNDPWR #PWR0164
+L GNDPWR #PWR0167
 U 1 1 4E93CEC2
 P 4500 2050
-F 0 "#PWR0164" H 4500 2100 40  0001 C CNN
+F 0 "#PWR0167" H 4500 2100 40  0001 C CNN
 F 1 "GNDPWR" H 4500 1970 40  0000 C CNN
 	1    4500 2050
@@
 	1    4050 1550
 	0    -1   -1   0
-$EndComp
-$Comp
-L C C79
-U 1 1 4E93CE80
-P 3600 1850
-F 0 "C79" H 3650 1950 50  0000 L CNN
-F 1 "63uf" H 3800 1950 50  0000 L CNN
-F 2 "2x200mil" H 3850 1850 60  0000 C CNN
-	1    3600 1850
-	1    0    0    -1
 $EndComp
 Text Notes 1600 5350 0    60   ~ 0
@@
 $EndComp
 $Comp
-L GNDPWR #PWR0165
+L GNDPWR #PWR0168
 U 1 1 4E93CAED
 P 5400 5400
-F 0 "#PWR0165" H 5400 5450 40  0001 C CNN
+F 0 "#PWR0168" H 5400 5450 40  0001 C CNN
 F 1 "GNDPWR" H 5400 5320 40  0000 C CNN
 	1    5400 5400
@@
 $EndComp
 $Comp
-L GND #PWR0166
+L GND #PWR0169
 U 1 1 4E93CA59
 P 7150 6350
-F 0 "#PWR0166" H 7150 6350 30  0001 C CNN
+F 0 "#PWR0169" H 7150 6350 30  0001 C CNN
 F 1 "GND" H 7150 6280 30  0001 C CNN
 	1    7150 6350
@@
 $EndComp
 $Comp
-L GND #PWR0167
+L GND #PWR0170
 U 1 1 4E93C3ED
 P 8800 2450
-F 0 "#PWR0167" H 8800 2450 30  0001 C CNN
+F 0 "#PWR0170" H 8800 2450 30  0001 C CNN
 F 1 "GND" H 8800 2380 30  0001 C CNN
 	1    8800 2450
@@
 $EndComp
 $Comp
-L GND #PWR0168
+L GND #PWR0171
 U 1 1 4E93C3EA
 P 8400 2450
-F 0 "#PWR0168" H 8400 2450 30  0001 C CNN
+F 0 "#PWR0171" H 8400 2450 30  0001 C CNN
 F 1 "GND" H 8400 2380 30  0001 C CNN
 	1    8400 2450
@@
 VC
 $Comp
-L GNDPWR #PWR0169
+L GNDPWR #PWR0172
 U 1 1 4E93C297
 P 6300 3900
-F 0 "#PWR0169" H 6300 3950 40  0001 C CNN
+F 0 "#PWR0172" H 6300 3950 40  0001 C CNN
 F 1 "GNDPWR" H 6300 3820 40  0000 C CNN
 	1    6300 3900
@@
 $EndComp
 $Comp
-L GNDPWR #PWR0170
+L GNDPWR #PWR0173
 U 1 1 4E93C0DB
 P 6200 2200
-F 0 "#PWR0170" H 6200 2250 40  0001 C CNN
+F 0 "#PWR0173" H 6200 2250 40  0001 C CNN
 F 1 "GNDPWR" H 6200 2120 40  0000 C CNN
 	1    6200 2200
@@
 VB
 $Comp
-L GNDPWR #PWR0171
+L GNDPWR #PWR0174
 U 1 1 4E93BDFD
 P 4600 4650
-F 0 "#PWR0171" H 4600 4700 40  0001 C CNN
+F 0 "#PWR0174" H 4600 4700 40  0001 C CNN
 F 1 "GNDPWR" H 4600 4570 40  0000 C CNN
 	1    4600 4650
@@
 $EndComp
 $Comp
-L GNDPWR #PWR0172
+L GNDPWR #PWR0175
 U 1 1 4E93BA9D
 P 5850 3800
-F 0 "#PWR0172" H 5850 3850 40  0001 C CNN
+F 0 "#PWR0175" H 5850 3850 40  0001 C CNN
 F 1 "GNDPWR" H 5850 3720 40  0000 C CNN
 	1    5850 3800
@@
 $EndComp
 $Comp
-L GNDPWR #PWR0173
+L GNDPWR #PWR0176
 U 1 1 4E93B6D0
 P 4300 3300
-F 0 "#PWR0173" H 4300 3350 40  0001 C CNN
+F 0 "#PWR0176" H 4300 3350 40  0001 C CNN
 F 1 "GNDPWR" H 4300 3220 40  0000 C CNN
 	1    4300 3300
@@
 $EndComp
 $Comp
-L GNDPWR #PWR0174
+L GNDPWR #PWR0177
 U 1 1 4E93B525
 P 2400 3050
-F 0 "#PWR0174" H 2400 3100 40  0001 C CNN
+F 0 "#PWR0177" H 2400 3100 40  0001 C CNN
 F 1 "GNDPWR" H 2400 2970 40  0000 C CNN
 	1    2400 3050

Commit message: finished parts order to digi-key. not much to do now but wait and/or build up an old board..
Parts:
- R129: value 7.15k -> 7k
Changed lines of the file:
@@
-EESchema Schematic File Version 2  date Thu 20 Oct 2011 05:59:00 PM EDT
+EESchema Schematic File Version 2  date Sat 22 Oct 2011 02:30:34 PM EDT
 LIBS:power
 LIBS:device
@@
 Sheet 2 3
 Title ""
-Date "20 oct 2011"
+Date "22 oct 2011"
 Rev ""
 Comp ""
@@
 	1    0    0    -1
 $EndComp
-Text Notes 3400 2300 0    60   ~ 0
-493-1665-ND
 $Comp
 L C C80
@@
 P 7400 5300
 F 0 "R129" V 7480 5300 50  0000 C CNN
-F 1 "7.15k" V 7400 5300 50  0000 C CNN
+F 1 "7k" V 7400 5300 50  0000 C CNN
 F 2 "0402" V 7530 5250 60  0001 C CNN
 	1    7400 5300
