File: emg_dsp/stage10/stage10.sch (KiCad schematic (older format))
At the start: 226 parts, among them U1 RS232_CON, U10 EN_VDD, U11 USBLC6, U12 ABM10XTAL-24, U13 BF527, U14 MIC5365-2.5, U15 SST25VF040B, U16 ADSP_JTAG_CON, U17 LAN8710A, U18 74LCX541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

Commit message: cleaned up firingrate.h -- not sure why this was not commited!
Other:
- moved on the sheet: C1, C10, C11, C12, C13, C14, C15, C16, C17, C18, C19, C2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
