File: emg_dsp/stage9/stage9.sch (KiCad schematic (older format))
At the start: 101 parts, among them U1 VEE, U10 74LCX541, U11 MAX6711Z, U12 ANTENNA, U13 TESTCON, U2 74LCX541, U3 9X100, U4 TPS62410, U5 ABM10XTAL-16, U6 BF532-160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

Commit message: that was a quick mod! now need to update the board & update stage7 accordingly.
Parts:
- removed C33: 33pf, 0402, symbol C
- removed C34, C5: 0.1uf, 0402, symbol C
- removed D1, D2, D3, D4, D5, D6, D7, D8: LED, 0603, symbol LED
- removed R1, R2, R3, R4, R5, R6, R7, R8: 50, 0402, symbol R
- removed R10, R11, R12, R9: 200, 0402, symbol R
- removed R18, R24, R25: 10k, 0402, symbol R
- removed TP1: PF0_nRF-CE, TP, symbol TP
- removed TP2: PF1_nRF-CSN, TP, symbol TP
- removed TP3: PF3_nRF-IRQ, TP, symbol TP
- removed TP4: PF4, TP, symbol TP
- removed TP5: PF8_STEP, TP, symbol TP
- removed TP6: RSCLK0, TP, symbol TP
- removed TP7: RFS0, TP, symbol TP
- removed TP8: DR0PRI, TP, symbol TP
- removed U10, U2: 74LCX541, TSSOP-20, symbol 74LCX541
- removed U13: TESTCON, 7x100mil, symbol TESTCON
- removed U7: ADSP_JTAG_CON, 7x2x100, symbol ADSP_JTAG_CON
- added C67: 1uf, 0402, symbol C
- added D1: 475-2558-1, 0603, symbol D
- added R79, R80: 200, 0402, symbol R
- R14: value 700k -> 725k
- R15: value 115k -> 160k
Connections:
- net labels added: MR
- wire segments 214 -> 157
- no-connect marks 8 -> 7
Other:
- note added: "0.95V"
- note added: "2.8V"
- note added: "_cs needs 33pf cap prior buf\ninputs should be driven through R 200"
- note added: "in"
- note added: "out"
- note added: "the blackfin does not have 5v tolerant inputs\nsource = 3.3V, Vdd=2.7V here, should be ok"
- note removed: "0.85V"
- note removed: "2.7V"
- note removed: "high-speed serial output"
- note removed: "the blackfin does not have 5v tolerant inputs"
- moved on the sheet: R30, U11, U3

Commit message: revised.
Parts:
- added U46: 9X100, omnetics_9, symbol 9X100
- R15: value 160k -> 165k
Connections:
- wire segments 157 -> 159

Commit message: word, schematics for 9/10 are close to done. start changing the boards...
Parts:
- removed R19, R20, R22, R27: 33, 0402, symbol R
- added R81, R82: 22k, 0402, symbol R
- D1: value 475-2558-1 -> 475-2558
- R17, R21: value 50k -> 22k
- R30: value 10k -> 22k
Connections:
- wire segments 159 -> 161

Commit message: working on stage9.
Parts:
- removed D1: 475-2558, 0603, symbol D
- removed TP10: 28, TP, symbol TP
- removed TP9: 08, TP, symbol TP
- added D?: LED, symbol LED
Changed lines of the file:
@@
-EESchema Schematic File Version 2  date Tue 11 Oct 2011 04:25:11 PM EDT
+EESchema Schematic File Version 2  date Wed 12 Oct 2011 11:50:05 PM EDT
 LIBS:power
 LIBS:device
@@
 Sheet 1 5
 Title "Stage 4 / Copyright 2010 Timothy L Hanson "
-Date "11 oct 2011"
+Date "13 oct 2011"
 Rev ""
 Comp "This design is free: redistribute or modify under the GPL v. 3 or later"
@@
 Comment4 ""
 $EndDescr
+$Comp
+L LED D?
+U 1 1 4E965FEA
+P 13950 4350
+F 0 "D?" H 13950 4450 50  0000 C CNN
+F 1 "LED" H 13950 4250 50  0000 C CNN
+	1    13950 4350
+	1    0    0    -1
+$EndComp
 Wire Wire Line
 	10750 2150 11250 2150
@@
 	1    14400 4350
 	0    1    1    0
-$EndComp
-$Comp
-L D D1
-U 1 1 4E8F745C
-P 13950 4350
-F 0 "D1" H 13950 4500 60  0000 C CNN
-F 1 "475-2558" H 13950 4150 60  0000 C CNN
-F 2 "0603" H 14150 4250 50  0000 C CNN
-	1    13950 4350
-	-1   0    0    1
 $EndComp
 $Comp
@@
 Text Notes 4650 8250 0    60   ~ 0
 TPS62420 also ok
-$Comp
-L TP TP9
-U 1 1 4C2A4FF1
-P 7050 7800
-F 0 "TP9" H 7150 7800 60  0000 C CNN
-F 1 "08" H 7300 7800 60  0000 C CNN
-F 2 "TP" H 7000 7900 60  0000 C CNN
-	1    7050 7800
-	1    0    0    -1
-$EndComp
-$Comp
-L TP TP10
-U 1 1 4C2A4FCD
-P 7100 9300
-F 0 "TP10" H 7200 9300 60  0000 C CNN
-F 1 "28" H 7350 9300 60  0000 C CNN
-F 2 "TP" H 7050 9400 60  0000 C CNN
-	1    7100 9300
-	1    0    0    -1
-$EndComp
 NoConn ~ 7750 3000
 Text Label 11350 3950 2    60   ~ 0
@@
 Text Label 9450 1700 2    60   ~ 0
 PF1
-Text Notes 7100 9250 0    60   ~ 0
+Text Notes 6950 9300 0    60   ~ 0
 0.95V
-Text Notes 7050 7650 0    60   ~ 0
+Text Notes 6900 7650 0    60   ~ 0
 2.8V
 $Comp

Commit message: boards done!! now need to produce gerbers etc.
Parts:
- added C68: 0.1uf, 0402, symbol C
- D1: renamed from D?; footprint (none) -> D0603
Connections:
- net GND: now also C68.2
- net VDD: now also C68.1
Changed lines of the file:
@@
-EESchema Schematic File Version 2  date Wed 12 Oct 2011 11:50:05 PM EDT
+EESchema Schematic File Version 2  date Thu 13 Oct 2011 06:49:24 PM EDT
 LIBS:power
 LIBS:device
@@
 Comment4 ""
 $EndDescr
-$Comp
-L LED D?
-U 1 1 4E965FEA
-P 13950 4350
-F 0 "D?" H 13950 4450 50  0000 C CNN
-F 1 "LED" H 13950 4250 50  0000 C CNN
-	1    13950 4350
-	1    0    0    -1
-$EndComp
+Connection ~ 11100 1150
+Wire Wire Line
+	11450 1150 8000 1150
 Wire Wire Line
 	10750 2150 11250 2150
@@
 	11900 1950 11900 2050
 Connection ~ 10700 750
-Wire Wire Line
-	11100 750  8000 750
 Wire Wire Line
 	3950 8650 3950 9450
@@
 Wire Wire Line
 	10750 2050 11250 2050
-Wire Wire Line
-	11100 1150 8000 1150
 Connection ~ 10700 1150
 Wire Wire Line
@@
 Wire Wire Line
 	10750 1950 11400 1950
+Wire Wire Line
+	11450 750  8000 750
+Connection ~ 11100 750
+$Comp
+L C C68
+U 1 1 4E973E32
+P 11450 950
+F 0 "C68" H 11500 1050 50  0000 L CNN
+F 1 "0.1uf" H 11500 850 50  0000 L CNN
+F 2 "0402" H 11550 1100 60  0000 C CNN
+	1    11450 950
+	1    0    0    -1
+$EndComp
+$Comp
+L LED D1
+U 1 1 4E965FEA
+P 13950 4350
+F 0 "D1" H 13950 4450 50  0000 C CNN
+F 1 "LED" H 13950 4250 50  0000 C CNN
+F 2 "D0603" H 13900 4500 60  0001 C CNN
+	1    13950 4350
+	1    0    0    -1
+$EndComp
 $Comp
 L GND #PWR01

Commit message: finished parts order to digi-key. not much to do now but wait and/or build up an old board..
Parts:
- C25: value 33nF -> 47nf
Changed lines of the file:
@@
-EESchema Schematic File Version 2  date Thu 13 Oct 2011 06:49:24 PM EDT
+EESchema Schematic File Version 2  date Sat 22 Oct 2011 01:28:52 PM EDT
 LIBS:power
 LIBS:device
@@
 Sheet 1 5
 Title "Stage 4 / Copyright 2010 Timothy L Hanson "
-Date "13 oct 2011"
+Date "22 oct 2011"
 Rev ""
 Comp "This design is free: redistribute or modify under the GPL v. 3 or later"
@@
 P 12050 5700
 F 0 "C25" H 12100 5800 50  0000 L CNN
-F 1 "33nF" H 12100 5600 50  0000 L CNN
+F 1 "47nf" H 12100 5600 50  0000 L CNN
 F 2 "0402" H 12150 5850 60  0000 C CNN
 	1    12050 5700

Commit message: cleaned up firingrate.h -- not sure why this was not commited!
Other:
- moved on the sheet: C1, C10, C11, C12, C13, C14, C15, C16, C17, C18, C19, C2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
