File: emg_dsp/stage11/analog.sch (KiCad schematic (older format))
At the start: 15 parts, among them U35 OMNETICS_36, U40 ADCS7476, U45 RHA2132

Commit message: gtkclient_tdt is still in tree-conflict. uff.
Changed lines of the file:
@@
-EESchema Schematic File Version 2  date Thu 07 Nov 2013 11:53:21 PM PST
+EESchema Schematic File Version 2  date Tue 12 Nov 2013 12:54:21 PM PST
 LIBS:power
 LIBS:device
@@
 $Descr User 16000 12000
 encoding utf-8
-Sheet 5 5
+Sheet 4 5
 Title "Stage 4 / Copyright 2010 Timothy L Hanson "
-Date "8 nov 2013"
+Date "12 nov 2013"
 Rev ""
 Comp "This design is free: redistribute or modify under the GPL v. 3 or later"
@@
 AR Path="/4D2BA3F8/4D2CD1D7" Ref="U43"  Part="1"
 AR Path="/4D2BA3AC/4D2CD1D7" Ref="U42"  Part="1"
-F 0 "U42" H 7650 3750 60  0000 C CNN
+F 0 "U43" H 7650 3750 60  0000 C CNN
 F 1 "RHA2132" H 7650 3900 60  0000 C CNN
 F 2 "QFN-56" H 7650 3600 60  0000 C CNN
@@
 AR Path="/4D2BA3F8/4D2CA6B7" Ref="R46"  Part="1"
 AR Path="/4D2BA3AC/4D2CA6B7" Ref="R34"  Part="1"
-F 0 "R34" V 4930 6200 50  0000 C CNN
+F 0 "R46" V 4930 6200 50  0000 C CNN
 F 1 "0" V 4850 6200 50  0000 C CNN
 F 2 "0201" V 4750 6200 60  0000 C CNN
@@
 AR Path="/4D2BA3F8/4D2CA69A" Ref="R43"  Part="1"
 AR Path="/4D2BA3AC/4D2CA69A" Ref="R31"  Part="1"
-F 0 "R31" V 3780 3550 50  0000 C CNN
+F 0 "R43" V 3780 3550 50  0000 C CNN
 F 1 "0" V 3700 3550 50  0000 C CNN
 F 2 "0201" V 3600 3550 60  0000 C CNN
@@
 AR Path="/4D2BA3F8/4D2B9CA3" Ref="R49"  Part="1"
 AR Path="/4D2BA3AC/4D2B9CA3" Ref="R37"  Part="1"
-F 0 "R37" V 9030 4200 50  0000 C CNN
+F 0 "R49" V 9030 4200 50  0000 C CNN
 F 1 "15k" V 8950 4200 50  0000 C CNN
 F 2 "0402" V 8950 4550 60  0000 C CNN
@@
 AR Path="/4D2BA3F8/4D2B9CA2" Ref="R51"  Part="1"
 AR Path="/4D2BA3AC/4D2B9CA2" Ref="R39"  Part="1"
-F 0 "R39" V 9030 4500 50  0000 C CNN
+F 0 "R51" V 9030 4500 50  0000 C CNN
 F 1 "7k" V 8950 4500 50  0000 C CNN
 F 2 "0402" V 8950 4850 60  0000 C CNN
@@
 AR Path="/4D2BA3F8/4D2B9CA1" Ref="#PWR0116"  Part="1"
 AR Path="/4D2BA3AC/4D2B9CA1" Ref="#PWR0141"  Part="1"
-F 0 "#PWR0141" H 9200 4200 30  0001 C CNN
+F 0 "#PWR0116" H 9200 4200 30  0001 C CNN
 F 1 "GND" H 9200 4130 30  0001 C CNN
 	1    9200 4200
@@
 AR Path="/4D2BA3F8/4D2B9CA0" Ref="#PWR0117"  Part="1"
 AR Path="/4D2BA3AC/4D2B9CA0" Ref="#PWR0142"  Part="1"
-F 0 "#PWR0142" H 9200 4350 30  0001 C CNN
+F 0 "#PWR0117" H 9200 4350 30  0001 C CNN
 F 1 "GND" H 9200 4280 30  0001 C CNN
 	1    9200 4350
@@
 AR Path="/4D2BA3F8/4D2B9C9F" Ref="R50"  Part="1"
 AR Path="/4D2BA3AC/4D2B9C9F" Ref="R38"  Part="1"
-F 0 "R38" V 9030 4350 50  0000 C CNN
+F 0 "R50" V 9030 4350 50  0000 C CNN
 F 1 "25.2k" V 8950 4350 50  0000 C CNN
 F 2 "0402" V 8950 4700 60  0000 C CNN
@@
 AR Path="/4D2BA3F8/4D2B9C9E" Ref="#PWR0118"  Part="1"
 AR Path="/4D2BA3AC/4D2B9C9E" Ref="#PWR0143"  Part="1"
-F 0 "#PWR0143" H 9200 4500 30  0001 C CNN
+F 0 "#PWR0118" H 9200 4500 30  0001 C CNN
 F 1 "GND" H 9200 4430 30  0001 C CNN
 	1    9200 4500
@@
 AR Path="/4D2BA3F8/4D2B9C3D" Ref="#PWR0119"  Part="1"
 AR Path="/4D2BA3AC/4D2B9C3D" Ref="#PWR0144"  Part="1"
-F 0 "#PWR0144" H 8250 4100 30  0001 C CNN
+F 0 "#PWR0119" H 8250 4100 30  0001 C CNN
 F 1 "GND" H 8250 4030 30  0001 C CNN
 	1    8250 4100
@@
 AR Path="/4D2BA3F8/4D2B9BE0" Ref="#PWR0120"  Part="1"
 AR Path="/4D2BA3AC/4D2B9BE0" Ref="#PWR0145"  Part="1"
-F 0 "#PWR0145" H 8300 4700 30  0001 C CNN
+F 0 "#PWR0120" H 8300 4700 30  0001 C CNN
 F 1 "GND" H 8300 4630 30  0001 C CNN
 	1    8300 4700
@@
 AR Path="/4D2BA3F8/4D2B9BCF" Ref="#PWR0121"  Part="1"
 AR Path="/4D2BA3AC/4D2B9BCF" Ref="#PWR0146"  Part="1"
-F 0 "#PWR0146" H 8250 6400 30  0001 C CNN
+F 0 "#PWR0121" H 8250 6400 30  0001 C CNN
 F 1 "GND" H 8250 6330 30  0001 C CNN
 	1    8250 6400
@@
 AR Path="/4D2BA3F8/4D2B9B34" Ref="#PWR0122"  Part="1"
 AR Path="/4D2BA3AC/4D2B9B34" Ref="#PWR0147"  Part="1"
-F 0 "#PWR0147" H 8900 5500 30  0001 C CNN
+F 0 "#PWR0122" H 8900 5500 30  0001 C CNN
 F 1 "GND" H 8900 5430 30  0001 C CNN
 	1    8900 5500
@@
 AR Path="/4D2BA3F8/4D2B9B31" Ref="#PWR0123"  Part="1"
 AR Path="/4D2BA3AC/4D2B9B31" Ref="#PWR0148"  Part="1"
-F 0 "#PWR0148" H 8900 4000 30  0001 C CNN
+F 0 "#PWR0123" H 8900 4000 30  0001 C CNN
 F 1 "GND" H 8900 3930 30  0001 C CNN
 	1    8900 4000
@@
 AR Path="/4D2BA3F8/4D2B9B2B" Ref="C47"  Part="1"
 AR Path="/4D2BA3AC/4D2B9B2B" Ref="C39"  Part="1"
-F 0 "C39" H 8700 4100 50  0000 L CNN
+F 0 "C47" H 8700 4100 50  0000 L CNN
 F 1 "0.1uf" H 8700 3900 50  0000 L CNN
 F 2 "0402" H 8800 3800 60  0000 C CNN
@@
 AR Path="/4D2BA3F8/4D2B9B24" Ref="C48"  Part="1"
 AR Path="/4D2BA3AC/4D2B9B24" Ref="C40"  Part="1"
-F 0 "C40" H 8700 5600 50  0000 L CNN
+F 0 "C48" H 8700 5600 50  0000 L CNN
 F 1 "0.1uf" H 8700 5400 50  0000 L CNN
 F 2 "0402" H 8800 5300 60  0000 C CNN
@@
 AR Path="/4D2BA3F8/4D2B8F4C" Ref="#PWR0124"  Part="1"
 AR Path="/4D2BA3AC/4D2B8F4C" Ref="#PWR0149"  Part="1"
-F 0 "#PWR0149" H 8400 3900 30  0001 C CNN
+F 0 "#PWR0124" H 8400 3900 30  0001 C CNN
 F 1 "GND" H 8400 3830 30  0001 C CNN
 	1    8400 3900
@@
 AR Path="/4D2BA3F8/4D2B8EB0" Ref="R45"  Part="1"
 AR Path="/4D2BA3AC/4D2B8EB0" Ref="R33"  Part="1"
-F 0 "R33" V 4680 5950 50  0000 C CNN
+F 0 "R45" V 4680 5950 50  0000 C CNN
 F 1 "0" V 4600 5950 50  0000 C CNN
 F 2 "0201" V 4750 5950 60  0000 C CNN
@@
 AR Path="/4D2BA3F8/4D2B8E82" Ref="R44"  Part="1"
 AR Path="/4D2BA3AC/4D2B8E82" Ref="R32"  Part="1"
-F 0 "R32" V 4030 3800 50  0000 C CNN
+F 0 "R44" V 4030 3800 50  0000 C CNN
 F 1 "0" V 3950 3800 50  0000 C CNN
 F 2 "0201" V 3850 3800 60  0000 C CNN
@@
 AR Path="/4D2BA3F8/4D2B89FA" Ref="U26"  Part="1"
 AR Path="/4D2BA3AC/4D2B89FA" Ref="U19"  Part="1"
-F 0 "U19" H 10500 4200 60  0000 C CNN
+F 0 "U26" H 10500 4200 60  0000 C CNN
 F 1 "ADCS7476" H 10550 4750 60  0000 C CNN
 F 2 "SOT-23-6" H 10600 4100 60  0000 C CNN
@@
 AR Path="/4D2BA3F8/4D2B89F9" Ref="#PWR0125"  Part="1"
 AR Path="/4D2BA3AC/4D2B89F9" Ref="#PWR0150"  Part="1"
-F 0 "#PWR0150" H 10200 4450 30  0001 C CNN
+F 0 "#PWR0125" H 10200 4450 30  0001 C CNN
 F 1 "GND" H 10200 4380 30  0001 C CNN
 	1    10200 4450
@@
 AR Path="/4D2BA3F8/4D2B89F8" Ref="C49"  Part="1"
 AR Path="/4D2BA3AC/4D2B89F8" Ref="C41"  Part="1"
-F 0 "C41" H 10050 5150 50  0000 L CNN
+F 0 "C49" H 10050 5150 50  0000 L CNN
 F 1 "0.1uf" H 10050 4950 50  0000 L CNN
 F 2 "0402" H 10250 5050 60  0000 C CNN
@@
 AR Path="/4D2BA3F8/4D2B89F7" Ref="#PWR0126"  Part="1"
 AR Path="/4D2BA3AC/4D2B89F7" Ref="#PWR0151"  Part="1"
-F 0 "#PWR0151" H 10000 5300 30  0001 C CNN
+F 0 "#PWR0126" H 10000 5300 30  0001 C CNN
 F 1 "GND" H 10000 5230 30  0001 C CNN
 	1    10000 5300
@@
 AR Path="/4D2BA3F8/4D2B89F6" Ref="R53"  Part="1"
 AR Path="/4D2BA3AC/4D2B89F6" Ref="R41"  Part="1"
-F 0 "R41" V 11380 4450 50  0000 C CNN
+F 0 "R53" V 11380 4450 50  0000 C CNN
 F 1 "200" V 11300 4450 50  0000 C CNN
 F 2 "0402" V 11200 4450 60  0000 C CNN
@@
 AR Path="/4D2BA3F8/4D2B89F5" Ref="C50"  Part="1"
 AR Path="/4D2BA3AC/4D2B89F5" Ref="C42"  Part="1"
-F 0 "C42" H 10350 5150 50  0000 L CNN
+F 0 "C50" H 10350 5150 50  0000 L CNN
 F 1 "2.2uf" H 10350 4950 50  0000 L CNN
 F 2 "0402" H 10400 5200 60  0000 C CNN
@@
 AR Path="/4D2BA3F8/4CA0ED5B" Ref="#PWR0130"  Part="1"
 AR Path="/4D2BA3AC/4CA0ED5B" Ref="#PWR0155"  Part="1"
-F 0 "#PWR0155" H 4250 6100 30  0001 C CNN
+F 0 "#PWR0130" H 4250 6100 30  0001 C CNN
 F 1 "GND" H 4250 6030 30  0001 C CNN
 	1    4250 6100
@@
 AR Path="/4D2BA3F8/4CA0ED5A" Ref="#PWR0131"  Part="1"
 AR Path="/4D2BA3AC/4CA0ED5A" Ref="#PWR0156"  Part="1"
-F 0 "#PWR0156" H 4250 3750 30  0001 C CNN
+F 0 "#PWR0131" H 4250 3750 30  0001 C CNN
 F 1 "GND" H 4250 3680 30  0001 C CNN
 	1    4250 3750
@@
 AR Path="/4D2BA3F8/4913DE57" Ref="U21"  Part="1"
 AR Path="/4D2BA3AC/4913DE57" Ref="U14"  Part="1"
-F 0 "U14" H 4300 4600 60  0000 C CNN
+F 0 "U21" H 4300 4600 60  0000 C CNN
 F 1 "OMNETICS_36" H 4300 5800 60  0000 C CNN
 F 2 "omnetics_36_dual" V 4300 5050 60  0000 C CNN
