File: emg_dsp/stage11/stage11.sch (KiCad schematic (older format))
At the start: 71 parts, among them U1 VEE, U11 MAX6711Z, U12 ANTENNA, U3 9X100, U4 TPS62410, U46 9X100, U5 ABM10XTAL-16, U6 BF532-160, U8 NRF24L01, U9 SST25VF040B

Commit message: gtkclient_tdt is still in tree-conflict. uff.
Parts:
- added U?: 5X100, symbol 5X100
Connections:
- net GND: now also U?.3
- net RESET: now also U?.4
- net VCC: now also U?.2
- net VDD: now also U?.1
- new net CLKOUT: U?.5
Other:
- note added: "DNP Slave"
- note added: "signals to be shared between boards: \nground\n2.8v\n0.95v\nclock\nreset"

Commit message: starting pcb layout on stage11.
Parts:
- removed C17: 4.7pF, 0402, symbol C
- removed U?: 5X100, symbol 5X100
- added U13: 74LVC1G125, SC-70-5, symbol 74LVC1G125
- added U2: 7X100, 7x2mm, symbol 7X100
- gave numbers to parts that had none: 6
Connections:
- net CLKOUT: now also U13.4 (Y), U2.5
- net GND: now also U13.1 (_oe), U13.3 (GND), U2.3, U2.6
- net RESET: now also U2.4
- net VCC: now also U2.2
- net VDD: now also U13.5 (Vcc), U2.1
- net VEE: now also U2.7
- net at U5.3 (X2), U6.A11 (XTAL), U8.10 (XC1): now also U13.2 (A)
Other:
- note added: "input load 4pf"
- note added: "signals to be shared between boards: \n(not necessarily in this order)\nground\nVbat\n2.8v\n0.95v\nclock\nreset"
- note removed: "signals to be shared between boards: \nground\n2.8v\n0.95v\nclock\nreset"
